File: encoders.sch (KiCad schematic (older format))
At the start: 43 parts, among them U3 74HCT595, U7 PEL12D

Commit message: updates.
Parts:
- removed R1, R15, R22, R8: R, symbol R
- removed R10, R16, R17, R2, R23, R24, R3, R9: 10k, symbol R
- removed U?: 74HCT574_PWR, symbol 74HCT574_PWR
- added C6: C, symbol C
- added RN1: 628B103, symbol 628B
- added U8: 74HC245, symbol 74LS245
- gave numbers to parts that had none: 1
- renumbered C1 to CK11, C2 to CK12, C3 to CK21, C4 to CK22, C5 to CK31, C6 to CK32, C7 to CK41, C8 to CK42, U7 to ENC4, R5 to RK12, R6 to RK13, R4 to RK16, R7 to RK17, R12 to RK22, R13 to RK23, R11 to RK26, R14 to RK27, R19 to RK32, R20 to RK33, R18 to RK36, R21 to RK37, R26 to RK42, R27 to RK43, R25 to RK46, R28 to RK47
Connections:
- net labels added: VPULLUP
- net labels removed: BUF_CLK, SHIFT_OE
- wire segments 121 -> 148
Other:
- note added: "74245: pull DIR (A->B) high."
- note added: "FIXME: Actually use the right package!!!"
- note added: "Needs to be 5V/3V compatible --> use HCT"
- note added: "Resistor pack BI Technologies 628A103\navailable in 220 mil chip (SO16N but slightly wider),\n0.56€ @ Mouser.\nType A is 8 parallel (0.07€ a pop),\ntype B is pullup/downs (0.037€ a pop)."
- note removed: "Doesn't need to be a clocked reg,\ncould just be a tristate buffer."
- moved on the sheet: C11, CK11, CK12, CK21, CK22, CK31, CK32, CK41, CK42, ENC1, ENC2, ENC3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

Commit message: Minor
Parts:
- removed RN1: 628B103, symbol 628B
- added C16: CP1, symbol CP1
- added RPU1 (x4), RPU10, RPU11, RPU12, RPU5, RPU6, RPU7, RPU8, RPU9: 10k, symbol R
Connections:
- net +3.3V: now also C11.1, C6.1, C16.1
- net GND: now also C11.2, C6.2, C16.2
- net SW1: now also RPU10.2
- net SW2: now also RPU7.2
- net SW3: now also RPU1.2
- net SW4: now also RPU1.2
- net VPULLUP: now also RPU1.1, RPU1.1, RPU1.1, RPU1.1, RPU10.1, RPU11.1, RPU12.1, RPU5.1, RPU6.1, RPU7.1, RPU8.1, RPU9.1
- net at ENC4.A, RK46.2: now also RPU1.2
- net at ENC4.B, RK47.2: now also RPU1.2
- net at ENC3.B, RK37.2: now also RPU6.2
- net at ENC3.A, RK36.2: now also RPU5.2
- net at ENC2.A, RK26.2: now also RPU8.2
- net at ENC2.B, RK27.2: now also RPU9.2
- net at ENC1.B, RK17.2: now also RPU12.2
- net at ENC1.A, RK16.2: now also RPU11.2
Other:
- note added: "Dimension decoupling for shifting (MHz)\nplus LED power (64mA spikes)"
- note added: "Resistor pack BI Technologies 628A103\navailable in 220 mil chip (SO16N but slightly wider),\n0.56€ @ Mouser.\nType A is 8 parallel (0.07€ a pop),\ntype B is pullup/downs (0.037€ a pop).\nMouser 1206 resistors (667-ERJ-P08J103V) are 2€ for 100.\n0805 (667-ERJ-6GEYJ103V) are 1€ for 100."
- note removed: "FIXME: Actually use the right package!!!"
- note removed: "Resistor pack BI Technologies 628A103\navailable in 220 mil chip (SO16N but slightly wider),\n0.56€ @ Mouser.\nType A is 8 parallel (0.07€ a pop),\ntype B is pullup/downs (0.037€ a pop)."
- moved on the sheet: C11

Commit message: Updates
Parts:
- removed U3: 74HCT595, symbol 74HC595
- added U3: 74HC595-PWR, symbol 74HC595-PWR
Connections:
- net labels added: LED11, LED12, LED21, LED22, LED31, LED32, LED41, LED42
- wire segments 167 -> 166
