File: encoders.sch (KiCad schematic (older format))
At the start: 45 parts, among them U3 74HC595-PWR, U8 74HC245

Commit message: Package updates
Parts:
- removed C16: CP1, symbol CP1
- added C16: 10u, symbol C
- C11, C6: value C -> 100n
- RK12, RK22, RK32, RK42: value R -> 390
- RK13, RK23, RK33, RK43: value R -> 240
- RK16, RK17, RK26, RK27, RK36, RK37, RK46, RK47, RPU1, RPU10, RPU11, RPU12, RPU5, RPU6, RPU7, RPU8, RPU9: value 10k -> 20k
- U3: value 74HC595-PWR -> 74HCT595
Other:
- note added: "PEL12D green/red max 30mA. Vf is 3.2/1.95V.\nDriven at 8mA, resistors should be 225/381 ohms.\nterminal 2 is green, terminal 3 is red."
- moved on the sheet: C11

Commit message: Switch to shift registers. Routing.
Parts:
- removed U8: 74HC245, symbol 74LS245
- added U8: 74HC165, symbol 74LS165
Connections:
- net labels added: BTNSHIFT_IN, BTNSHIFT_OUT, BTN_CE, BTN_LOAD, LEDSHIFT_IN, LEDSHIFT_OUT, LED_LOAD, LED_OE
- net labels removed: BUF_OE, BUS_0, BUS_1, BUS_2, BUS_3, BUS_4, BUS_5, BUS_6, BUS_7, SHIFT_IN, SHIFT_LATCH, SHIFT_OUT
- wire segments 166 -> 173
- no-connect marks 0 -> 1
Other:
- note removed: "74245: pull DIR (A->B) high."
- moved on the sheet: C6

Commit message: Routing
Other:
- note removed: "Dimension decoupling for shifting (MHz)\nplus LED power (64mA spikes)"
- note removed: "Resistor pack BI Technologies 628A103\navailable in 220 mil chip (SO16N but slightly wider),\n0.56€ @ Mouser.\nType A is 8 parallel (0.07€ a pop),\ntype B is pullup/downs (0.037€ a pop).\nMouser 1206 resistors (667-ERJ-P08J103V) are 2€ for 100.\n0805 (667-ERJ-6GEYJ103V) are 1€ for 100."
Changed lines of the file:
@@
-EESchema Schematic File Version 2  date Tue 17 Apr 2012 08:42:54 PM CEST
+EESchema Schematic File Version 2  date Thu 19 Apr 2012 08:23:14 PM CEST
 LIBS:power
 LIBS:device
@@
 Sheet 3 5
 Title ""
-Date "17 apr 2012"
+Date "19 apr 2012"
 Rev ""
 Comp ""
@@
 	1    0    0    -1
 $EndComp
-Text Notes 1000 6250 0    60   ~ 0
-Dimension decoupling for shifting (MHz)\nplus LED power (64mA spikes)
 $Comp
 L R RPU12
@@
 	1    0    0    -1
 $EndComp
-Text Notes 5800 900  0    60   ~ 0
-Resistor pack BI Technologies 628A103\navailable in 220 mil chip (SO16N but slightly wider),\n0.56€ @ Mouser.\nType A is 8 parallel (0.07€ a pop),\ntype B is pullup/downs (0.037€ a pop).\nMouser 1206 resistors (667-ERJ-P08J103V) are 2€ for 100.\n0805 (667-ERJ-6GEYJ103V) are 1€ for 100.
 $Comp
 L +3.3V #PWR012
