File: encoders.sch (KiCad schematic (older format))
At the start: 45 parts, among them U3 74HCT595, U8 74HC165

Commit message: Chaotic changes.
Parts:
- removed RK16, RK17, RK26, RK27, RK36, RK37, RK46, RK47: 20k, symbol R
- CK11, CK12, CK21, CK22, CK31, CK32, CK41, CK42: value 10n -> DNP
Connections:
- wire segments 173 -> 165
Other:
- moved on the sheet: CK41, CK42

Commit message: Routing.
Parts:
- removed CK11, CK12, CK21, CK22, CK31, CK32, CK41, CK42: DNP, symbol C
Connections:
- wire segments 165 -> 149
Changed lines of the file:
@@
-EESchema Schematic File Version 2  date Sun 05 May 2013 06:02:32 PM CEST
+EESchema Schematic File Version 2  date Wed 08 May 2013 08:54:31 PM CEST
 LIBS:power
 LIBS:device
@@
 Sheet 10 10
 Title ""
-Date "5 may 2013"
+Date "8 may 2013"
 Rev ""
 Comp ""
@@
 Comment4 ""
 $EndDescr
-Connection ~ 7450 3700
-Connection ~ 7750 2050
-Wire Wire Line
-	7450 2350 7450 2250
-Wire Wire Line
-	7750 2750 7450 2750
-Wire Wire Line
-	7600 2800 7600 2750
-Connection ~ 7600 2750
-Wire Wire Line
-	7750 2350 7750 2050
-Wire Wire Line
-	7750 3800 7750 3500
-Connection ~ 7600 4200
-Wire Wire Line
-	7600 4250 7600 4200
-Wire Wire Line
-	7750 4200 7450 4200
-Wire Wire Line
-	7450 3800 7450 3700
-Connection ~ 7750 4950
-Wire Wire Line
-	7450 5250 7450 5150
-Wire Wire Line
-	7750 5650 7450 5650
-Wire Wire Line
-	7600 5700 7600 5650
-Connection ~ 7600 5650
-Wire Wire Line
-	7750 5250 7750 4950
-Wire Wire Line
-	7750 6750 7750 6450
+Wire Wire Line
+	6350 4950 8400 4950
 Wire Wire Line
 	6350 2250 8750 2250
@@
 Wire Wire Line
 	6350 6650 8700 6650
-Connection ~ 7750 6450
-Connection ~ 7450 6650
-Connection ~ 7600 7150
-Wire Wire Line
-	7600 7200 7600 7150
-Wire Wire Line
-	7750 7150 7450 7150
 Wire Wire Line
 	9000 5150 9000 5000
@@
 	8600 4500 9050 4500
 Wire Wire Line
-	8400 4300 8400 4950
+	8400 4950 8400 4300
 Wire Wire Line
 	8400 4300 9050 4300
@@
 	8600 6450 6350 6450
 Wire Wire Line
-	8400 4950 6350 4950
-Wire Wire Line
 	8650 3500 6350 3500
 Wire Wire Line
 	8850 2050 6350 2050
-Wire Wire Line
-	7450 6750 7450 6650
-Connection ~ 7450 5150
-Connection ~ 7450 2250
-Connection ~ 7750 3500
-$Comp
-L C CK11
-U 1 1 50CDFC59
-P 7450 2550
-F 0 "CK11" H 7500 2650 50  0000 L CNN
-F 1 "DNP" H 7500 2450 50  0000 L CNN
-	1    7450 2550
-	1    0    0    -1
-$EndComp
-$Comp
-L C CK12
-U 1 1 50CDFC58
-P 7750 2550
-F 0 "CK12" H 7800 2650 50  0000 L CNN
-F 1 "DNP" H 7800 2450 50  0000 L CNN
-	1    7750 2550
-	1    0    0    -1
-$EndComp
-$Comp
-L GND #PWR138
-U 1 1 50CDFC57
-P 7600 2800
-F 0 "#PWR138" H 7600 2800 30  0001 C CNN
-F 1 "GND" H 7600 2730 30  0001 C CNN
-	1    7600 2800
-	1    0    0    -1
-$EndComp
-$Comp
-L GND #PWR139
-U 1 1 50CDFC52
-P 7600 4250
-F 0 "#PWR139" H 7600 4250 30  0001 C CNN
-F 1 "GND" H 7600 4180 30  0001 C CNN
-	1    7600 4250
-	1    0    0    -1
-$EndComp
-$Comp
-L C CK22
-U 1 1 50CDFC51
-P 7750 4000
-F 0 "CK22" H 7800 4100 50  0000 L CNN
-F 1 "DNP" H 7800 3900 50  0000 L CNN
-	1    7750 4000
-	1    0    0    -1
-$EndComp
-$Comp
-L C CK21
-U 1 1 50CDFC50
-P 7450 4000
-F 0 "CK21" H 7500 4100 50  0000 L CNN
-F 1 "DNP" H 7500 3900 50  0000 L CNN
-	1    7450 4000
-	1    0    0    -1
-$EndComp
-$Comp
-L C CK31
-U 1 1 50CDFC43
-P 7450 5450
-F 0 "CK31" H 7500 5550 50  0000 L CNN
-F 1 "DNP" H 7500 5350 50  0000 L CNN
-	1    7450 5450
-	1    0    0    -1
-$EndComp
-$Comp
-L C CK32
-U 1 1 50CDFC42
-P 7750 5450
-F 0 "CK32" H 7800 5550 50  0000 L CNN
-F 1 "DNP" H 7800 5350 50  0000 L CNN
-	1    7750 5450
-	1    0    0    -1
-$EndComp
-$Comp
-L GND #PWR140
-U 1 1 50CDFC41
-P 7600 5700
-F 0 "#PWR140" H 7600 5700 30  0001 C CNN
-F 1 "GND" H 7600 5630 30  0001 C CNN
-	1    7600 5700
-	1    0    0    -1
-$EndComp
-$Comp
-L GND #PWR141
-U 1 1 4F7E095D
-P 7600 7200
-F 0 "#PWR141" H 7600 7200 30  0001 C CNN
-F 1 "GND" H 7600 7130 30  0001 C CNN
-	1    7600 7200
-	1    0    0    -1
-$EndComp
-$Comp
-L C CK42
-U 1 1 4F7E095C
-P 7750 6950
-F 0 "CK42" H 7800 7050 50  0000 L CNN
-F 1 "DNP" H 7800 6850 50  0000 L CNN
-	1    7750 6950
-	1    0    0    -1
-$EndComp
-$Comp
-L C CK41
-U 1 1 4F7E095B
-P 7450 6950
-F 0 "CK41" H 7500 7050 50  0000 L CNN
-F 1 "DNP" H 7500 6850 50  0000 L CNN
-	1    7450 6950
-	1    0    0    -1
-$EndComp
 NoConn ~ 10450 4000
 Text HLabel 8900 5150 3    60   Input ~ 0
@@
 $EndComp
 $Comp
-L +5V #PWR125
+L +5V #PWR0111
 U 1 1 4F834CB1
 P 1050 3200
-F 0 "#PWR125" H 1050 3290 20  0001 C CNN
+F 0 "#PWR0111" H 1050 3290 20  0001 C CNN
 F 1 "+5V" H 1050 3290 30  0000 C CNN
 	1    1050 3200
@@
 NXP 74HCT595 will source up to 8mA to each output\nand seems to be 5V/3V compatible.
 $Comp
-L +3.3V #PWR144
+L +3.3V #PWR0112
 U 1 1 4F829FD3
 P 10300 5550
-F 0 "#PWR144" H 10300 5510 30  0001 C CNN
+F 0 "#PWR0112" H 10300 5510 30  0001 C CNN
 F 1 "+3.3V" H 10300 5660 30  0000 C CNN
 	1    10300 5550
@@
 $EndComp
 $Comp
-L GND #PWR145
+L GND #PWR0113
 U 1 1 4F905A7B
 P 10300 6250
-F 0 "#PWR145" H 10300 6250 30  0001 C CNN
+F 0 "#PWR0113" H 10300 6250 30  0001 C CNN
 F 1 "GND" H 10300 6180 30  0001 C CNN
 	1    10300 6250
@@
 $EndComp
 $Comp
-L GND #PWR128
+L GND #PWR0114
 U 1 1 4F905A7A
 P 1850 7150
-F 0 "#PWR128" H 1850 7150 30  0001 C CNN
+F 0 "#PWR0114" H 1850 7150 30  0001 C CNN
 F 1 "GND" H 1850 7080 30  0001 C CNN
 	1    1850 7150
@@
 $EndComp
 $Comp
-L +5V #PWR127
+L +5V #PWR0115
 U 1 1 4F905A79
 P 1850 6500
-F 0 "#PWR127" H 1850 6590 20  0001 C CNN
+F 0 "#PWR0115" H 1850 6590 20  0001 C CNN
 F 1 "+5V" H 1850 6590 30  0000 C CNN
 	1    1850 6500
@@
 $EndComp
 $Comp
-L +3.3V #PWR142
+L +3.3V #PWR0116
 U 1 1 4F8131EC
 P 9450 3500
-F 0 "#PWR142" H 9450 3460 30  0001 C CNN
+F 0 "#PWR0116" H 9450 3460 30  0001 C CNN
 F 1 "+3.3V" H 9450 3610 30  0000 C CNN
 	1    9450 3500
@@
 $EndComp
 $Comp
-L GND #PWR143
+L GND #PWR0117
 U 1 1 4F8131C7
 P 9450 5250
-F 0 "#PWR143" H 9450 5250 30  0001 C CNN
+F 0 "#PWR0117" H 9450 5250 30  0001 C CNN
 F 1 "GND" H 9450 5180 30  0001 C CNN
 	1    9450 5250
@@
 Needs to be 5V/3V compatible --> use HCT
 $Comp
-L GND #PWR126
+L GND #PWR0118
 U 1 1 4F905A69
 P 1050 4700
-F 0 "#PWR126" H 1050 4700 30  0001 C CNN
+F 0 "#PWR0118" H 1050 4700 30  0001 C CNN
 F 1 "GND" H 1050 4630 30  0001 C CNN
 	1    1050 4700
@@
 $EndComp
 $Comp
-L GND #PWR132
+L GND #PWR0119
 U 1 1 4F905A68
 P 5150 5350
-F 0 "#PWR132" H 5150 5350 30  0001 C CNN
+F 0 "#PWR0119" H 5150 5350 30  0001 C CNN
 F 1 "GND" H 5150 5280 30  0001 C CNN
 	1    5150 5350
@@
 $EndComp
 $Comp
-L GND #PWR129
+L GND #PWR0120
 U 1 1 4F7E098D
 P 5150 2450
-F 0 "#PWR129" H 5150 2450 30  0001 C CNN
+F 0 "#PWR0120" H 5150 2450 30  0001 C CNN
 F 1 "GND" H 5150 2380 30  0001 C CNN
 	1    5150 2450
@@
 $EndComp
 $Comp
-L GND #PWR134
+L GND #PWR0121
 U 1 1 4F7E0987
 P 6600 2400
-F 0 "#PWR134" H 6600 2400 30  0001 C CNN
+F 0 "#PWR0121" H 6600 2400 30  0001 C CNN
 F 1 "GND" H 6600 2330 30  0001 C CNN
 	1    6600 2400
@@
 $EndComp
 $Comp
-L GND #PWR135
+L GND #PWR0122
 U 1 1 4F7E0976
 P 6600 3850
-F 0 "#PWR135" H 6600 3850 30  0001 C CNN
+F 0 "#PWR0122" H 6600 3850 30  0001 C CNN
 F 1 "GND" H 6600 3780 30  0001 C CNN
 	1    6600 3850
@@
 $EndComp
 $Comp
-L GND #PWR130
+L GND #PWR0123
 U 1 1 4F7E0970
 P 5150 3900
-F 0 "#PWR130" H 5150 3900 30  0001 C CNN
+F 0 "#PWR0123" H 5150 3900 30  0001 C CNN
 F 1 "GND" H 5150 3830 30  0001 C CNN
 	1    5150 3900
@@
 $EndComp
 $Comp
-L GND #PWR131
+L GND #PWR0124
 U 1 1 4F7E096D
 P 5150 5350
-F 0 "#PWR131" H 5150 5350 30  0001 C CNN
+F 0 "#PWR0124" H 5150 5350 30  0001 C CNN
 F 1 "GND" H 5150 5280 30  0001 C CNN
 	1    5150 5350
@@
 $EndComp
 $Comp
-L GND #PWR136
+L GND #PWR0125
 U 1 1 4F905A4E
 P 6600 5300
-F 0 "#PWR136" H 6600 5300 30  0001 C CNN
+F 0 "#PWR0125" H 6600 5300 30  0001 C CNN
 F 1 "GND" H 6600 5230 30  0001 C CNN
 	1    6600 5300
@@
 $EndComp
 $Comp
-L GND #PWR137
+L GND #PWR0126
 U 1 1 4F7E0956
 P 6600 6800
-F 0 "#PWR137" H 6600 6800 30  0001 C CNN
+F 0 "#PWR0126" H 6600 6800 30  0001 C CNN
 F 1 "GND" H 6600 6730 30  0001 C CNN
 	1    6600 6800
@@
 $EndComp
 $Comp
-L GND #PWR133
+L GND #PWR0127
 U 1 1 4F905A40
 P 5150 6850
-F 0 "#PWR133" H 5150 6850 30  0001 C CNN
+F 0 "#PWR0127" H 5150 6850 30  0001 C CNN
 F 1 "GND" H 5150 6780 30  0001 C CNN
 	1    5150 6850

Commit message: Finished board CAD?
Parts:
- RK13, RK23, RK33, RK43: value 240 -> 390
Changed lines of the file:
@@
-EESchema Schematic File Version 2  date Sat 01 Jun 2013 11:43:44 AM CEST
+EESchema Schematic File Version 2  date Sat 08 Jun 2013 11:15:40 AM CEST
 LIBS:power
 LIBS:device
@@
 Sheet 10 10
 Title ""
-Date "1 jun 2013"
+Date "8 jun 2013"
 Rev ""
 Comp ""
@@
 $EndComp
 $Comp
-L +5V #PWR108
+L +5V #PWR0113
 U 1 1 4F834CB1
 P 1050 3200
-F 0 "#PWR108" H 1050 3290 20  0001 C CNN
+F 0 "#PWR0113" H 1050 3290 20  0001 C CNN
 F 1 "+5V" H 1050 3290 30  0000 C CNN
 	1    1050 3200
@@
 NXP 74HCT595 will source up to 8mA to each output\nand seems to be 5V/3V compatible.
 $Comp
-L +3.3V #PWR123
+L +3.3V #PWR0114
 U 1 1 4F829FD3
 P 10300 5550
-F 0 "#PWR123" H 10300 5510 30  0001 C CNN
+F 0 "#PWR0114" H 10300 5510 30  0001 C CNN
 F 1 "+3.3V" H 10300 5660 30  0000 C CNN
 	1    10300 5550
@@
 $EndComp
 $Comp
-L GND #PWR124
+L GND #PWR0115
 U 1 1 4F905A7B
 P 10300 6250
-F 0 "#PWR124" H 10300 6250 30  0001 C CNN
+F 0 "#PWR0115" H 10300 6250 30  0001 C CNN
 F 1 "GND" H 10300 6180 30  0001 C CNN
 	1    10300 6250
@@
 $EndComp
 $Comp
-L GND #PWR111
+L GND #PWR0116
 U 1 1 4F905A7A
 P 1850 7150
-F 0 "#PWR111" H 1850 7150 30  0001 C CNN
+F 0 "#PWR0116" H 1850 7150 30  0001 C CNN
 F 1 "GND" H 1850 7080 30  0001 C CNN
 	1    1850 7150
@@
 $EndComp
 $Comp
-L +5V #PWR110
+L +5V #PWR0117
 U 1 1 4F905A79
 P 1850 6500
-F 0 "#PWR110" H 1850 6590 20  0001 C CNN
+F 0 "#PWR0117" H 1850 6590 20  0001 C CNN
 F 1 "+5V" H 1850 6590 30  0000 C CNN
 	1    1850 6500
@@
 $EndComp
 $Comp
-L +3.3V #PWR121
+L +3.3V #PWR0118
 U 1 1 4F8131EC
 P 9450 3500
-F 0 "#PWR121" H 9450 3460 30  0001 C CNN
+F 0 "#PWR0118" H 9450 3460 30  0001 C CNN
 F 1 "+3.3V" H 9450 3610 30  0000 C CNN
 	1    9450 3500
@@
 $EndComp
 $Comp
-L GND #PWR122
+L GND #PWR0119
 U 1 1 4F8131C7
 P 9450 5250
-F 0 "#PWR122" H 9450 5250 30  0001 C CNN
+F 0 "#PWR0119" H 9450 5250 30  0001 C CNN
 F 1 "GND" H 9450 5180 30  0001 C CNN
 	1    9450 5250
@@
 Needs to be 5V/3V compatible --> use HCT
 $Comp
-L GND #PWR109
+L GND #PWR0120
 U 1 1 4F905A69
 P 1050 4700
-F 0 "#PWR109" H 1050 4700 30  0001 C CNN
+F 0 "#PWR0120" H 1050 4700 30  0001 C CNN
 F 1 "GND" H 1050 4630 30  0001 C CNN
 	1    1050 4700
@@
 $EndComp
 $Comp
-L GND #PWR115
+L GND #PWR0121
 U 1 1 4F905A68
 P 5150 5350
-F 0 "#PWR115" H 5150 5350 30  0001 C CNN
+F 0 "#PWR0121" H 5150 5350 30  0001 C CNN
 F 1 "GND" H 5150 5280 30  0001 C CNN
 	1    5150 5350
@@
 $EndComp
 $Comp
-L GND #PWR112
+L GND #PWR0122
 U 1 1 4F7E098D
 P 5150 2450
-F 0 "#PWR112" H 5150 2450 30  0001 C CNN
+F 0 "#PWR0122" H 5150 2450 30  0001 C CNN
 F 1 "GND" H 5150 2380 30  0001 C CNN
 	1    5150 2450
@@
 P 4850 2200
 F 0 "RK13" V 4930 2200 50  0000 C CNN
-F 1 "240" V 4850 2200 50  0000 C CNN
+F 1 "390" V 4850 2200 50  0000 C CNN
 	1    4850 2200
 	0    1    1    0
 $EndComp
 $Comp
-L GND #PWR117
+L GND #PWR0123
 U 1 1 4F7E0987
 P 6600 2400
-F 0 "#PWR117" H 6600 2400 30  0001 C CNN
+F 0 "#PWR0123" H 6600 2400 30  0001 C CNN
 F 1 "GND" H 6600 2330 30  0001 C CNN
 	1    6600 2400
@@
 $EndComp
 $Comp
-L GND #PWR118
+L GND #PWR0124
 U 1 1 4F7E0976
 P 6600 3850
-F 0 "#PWR118" H 6600 3850 30  0001 C CNN
+F 0 "#PWR0124" H 6600 3850 30  0001 C CNN
 F 1 "GND" H 6600 3780 30  0001 C CNN
 	1    6600 3850
@@
 P 4850 3650
 F 0 "RK23" V 4930 3650 50  0000 C CNN
-F 1 "240" V 4850 3650 50  0000 C CNN
+F 1 "390" V 4850 3650 50  0000 C CNN
 	1    4850 3650
 	0    1    1    0
@@
 $EndComp
 $Comp
-L GND #PWR113
+L GND #PWR0125
 U 1 1 4F7E0970
 P 5150 3900
-F 0 "#PWR113" H 5150 3900 30  0001 C CNN
+F 0 "#PWR0125" H 5150 3900 30  0001 C CNN
 F 1 "GND" H 5150 3830 30  0001 C CNN
 	1    5150 3900
@@
 $EndComp
 $Comp
-L GND #PWR114
+L GND #PWR0126
 U 1 1 4F7E096D
 P 5150 5350
-F 0 "#PWR114" H 5150 5350 30  0001 C CNN
+F 0 "#PWR0126" H 5150 5350 30  0001 C CNN
 F 1 "GND" H 5150 5280 30  0001 C CNN
 	1    5150 5350
@@
 P 4850 5100
 F 0 "RK33" V 4930 5100 50  0000 C CNN
-F 1 "240" V 4850 5100 50  0000 C CNN
+F 1 "390" V 4850 5100 50  0000 C CNN
 	1    4850 5100
 	0    1    1    0
 $EndComp
 $Comp
-L GND #PWR119
+L GND #PWR0127
 U 1 1 4F905A4E
 P 6600 5300
-F 0 "#PWR119" H 6600 5300 30  0001 C CNN
+F 0 "#PWR0127" H 6600 5300 30  0001 C CNN
 F 1 "GND" H 6600 5230 30  0001 C CNN
 	1    6600 5300
@@
 $EndComp
 $Comp
-L GND #PWR120
+L GND #PWR0128
 U 1 1 4F7E0956
 P 6600 6800
-F 0 "#PWR120" H 6600 6800 30  0001 C CNN
+F 0 "#PWR0128" H 6600 6800 30  0001 C CNN
 F 1 "GND" H 6600 6730 30  0001 C CNN
 	1    6600 6800
@@
 P 4850 6600
 F 0 "RK43" V 4930 6600 50  0000 C CNN
-F 1 "240" V 4850 6600 50  0000 C CNN
+F 1 "390" V 4850 6600 50  0000 C CNN
 	1    4850 6600
 	0    1    1    0
@@
 $EndComp
 $Comp
-L GND #PWR116
+L GND #PWR0129
 U 1 1 4F905A40
 P 5150 6850
-F 0 "#PWR116" H 5150 6850 30  0001 C CNN
+F 0 "#PWR0129" H 5150 6850 30  0001 C CNN
 F 1 "GND" H 5150 6780 30  0001 C CNN
 	1    5150 6850
