File: knobboard.sch (KiCad schematic (older format))
At the start: 10 parts

Commit message: Chaotic changes.
Changed lines of the file:
@@
-EESchema Schematic File Version 2  date Sat 15 Dec 2012 04:09:18 PM CET
+EESchema Schematic File Version 2  date Sun 16 Dec 2012 05:53:49 PM CET
 LIBS:power
 LIBS:device
@@
 Sheet 1 10
 Title ""
-Date "15 dec 2012"
+Date "16 dec 2012"
 Rev ""
 Comp ""
@@
 $EndDescr
 Wire Wire Line
+	3600 2000 2950 2000
+Wire Wire Line
+	3600 5350 2950 5350
+Wire Wire Line
+	3600 5150 2950 5150
+Wire Wire Line
+	3600 3100 2950 3100
+Wire Wire Line
+	3600 2900 2950 2900
+Wire Wire Line
+	2950 2200 3600 2200
+Wire Wire Line
+	3600 1900 2950 1900
+Wire Wire Line
+	6250 5400 6250 1150
+Wire Wire Line
+	6700 3200 6650 3200
+Wire Wire Line
+	6650 3200 6650 3850
+Wire Wire Line
+	6650 3850 8400 3850
+Wire Wire Line
+	8400 3850 8400 4700
+Wire Wire Line
+	8400 4700 8200 4700
+Wire Wire Line
+	8200 6000 8800 6000
+Wire Wire Line
+	8200 5800 8800 5800
+Wire Wire Line
+	8200 5700 8800 5700
+Wire Wire Line
+	8200 5600 8800 5600
+Wire Wire Line
+	8200 5500 8800 5500
+Wire Wire Line
+	6650 6400 6650 5700
+Wire Wire Line
+	6650 5700 6700 5700
+Connection ~ 6050 4600
+Wire Wire Line
+	6050 2200 6050 5900
+Wire Wire Line
+	6050 5900 6700 5900
+Connection ~ 6450 4300
+Wire Wire Line
+	6450 5600 6450 1350
+Wire Wire Line
+	6450 5600 6700 5600
+Wire Wire Line
+	6250 5400 6700 5400
+Wire Wire Line
+	6700 4700 6550 4700
+Wire Wire Line
+	6550 4700 6550 3750
+Wire Wire Line
+	6550 3750 8500 3750
+Wire Wire Line
+	8500 3750 8500 3550
+Wire Wire Line
+	8500 3550 8200 3550
+Connection ~ 6150 3300
+Wire Wire Line
+	6150 4500 6700 4500
+Connection ~ 6350 3000
+Wire Wire Line
+	6350 4200 6700 4200
+Connection ~ 6150 2100
+Wire Wire Line
+	6150 3300 6700 3300
+Wire Wire Line
+	6350 3000 6700 3000
+Wire Wire Line
+	8200 3450 8800 3450
+Wire Wire Line
+	8200 3100 8800 3100
+Wire Wire Line
+	8200 2900 8800 2900
+Wire Wire Line
+	5600 2500 5900 2500
+Connection ~ 6450 1900
+Wire Wire Line
+	6450 1350 8800 1350
+Wire Wire Line
+	6250 1150 8800 1150
+Wire Wire Line
+	5600 2200 6700 2200
+Wire Wire Line
+	5600 1900 6700 1900
+Wire Wire Line
+	5600 1700 6700 1700
+Wire Wire Line
+	8200 1900 8800 1900
+Wire Wire Line
+	8200 2100 8800 2100
+Wire Wire Line
+	8200 2000 8800 2000
+Wire Wire Line
+	8200 1800 8800 1800
+Wire Wire Line
+	6700 2300 5600 2300
+Wire Wire Line
+	6700 1800 5600 1800
+Wire Wire Line
+	6700 2100 5600 2100
+Connection ~ 6250 1700
+Wire Wire Line
+	8800 1250 6350 1250
+Connection ~ 6350 1800
+Wire Wire Line
+	8200 2250 8600 2250
+Wire Wire Line
+	8600 2250 8600 2550
+Wire Wire Line
+	8600 2550 5900 2550
+Wire Wire Line
+	5900 2550 5900 2500
+Wire Wire Line
+	6150 800  10350 800
+Wire Wire Line
+	6150 800  6150 2000
+Wire Wire Line
+	6150 2000 6700 2000
+Wire Wire Line
+	8800 3000 8200 3000
+Wire Wire Line
+	8800 3200 8200 3200
+Wire Wire Line
+	8200 2350 8500 2350
+Wire Wire Line
+	8500 2350 8500 2650
+Wire Wire Line
+	8500 2650 6550 2650
+Wire Wire Line
+	6550 2650 6550 3500
+Wire Wire Line
+	6550 3500 6700 3500
+Wire Wire Line
+	6250 2900 6700 2900
+Connection ~ 6250 2900
+Wire Wire Line
+	6450 3100 6700 3100
+Wire Wire Line
+	6050 3400 6700 3400
+Connection ~ 6050 2200
+Wire Wire Line
+	6250 4100 6700 4100
+Connection ~ 6250 4100
+Wire Wire Line
+	6450 4300 6700 4300
+Connection ~ 6450 3100
+Wire Wire Line
+	6700 4600 6050 4600
+Connection ~ 6050 3400
+Wire Wire Line
+	8200 4800 8550 4800
+Wire Wire Line
+	8550 4800 8550 5050
+Wire Wire Line
+	8550 5050 6550 5050
+Wire Wire Line
+	6550 5050 6550 6000
+Wire Wire Line
+	6550 6000 6700 6000
+Wire Wire Line
+	6700 5500 6350 5500
+Wire Wire Line
+	6350 5500 6350 1250
+Connection ~ 6350 4200
+Wire Wire Line
+	6700 5800 6150 5800
+Wire Wire Line
+	6150 5800 6150 2100
+Connection ~ 6150 4500
+Wire Wire Line
+	8200 6100 8350 6100
+Wire Wire Line
+	8200 4200 8800 4200
+Wire Wire Line
+	8200 4300 8800 4300
+Wire Wire Line
+	8200 4400 8800 4400
+Wire Wire Line
+	8200 4500 8800 4500
+Wire Wire Line
+	10350 800  10350 2500
+Wire Wire Line
+	10350 2500 10200 2500
+Wire Wire Line
+	10200 5000 10400 5000
+Wire Wire Line
+	10400 5000 10400 6950
+Wire Wire Line
+	10400 6950 5950 6950
+Wire Wire Line
+	5950 6950 5950 4400
+Wire Wire Line
+	5950 4400 6700 4400
+Wire Wire Line
+	2950 1700 3600 1700
+Wire Wire Line
+	3600 2100 2950 2100
+Wire Wire Line
+	2950 2800 3600 2800
+Wire Wire Line
+	2950 3000 3600 3000
+Wire Wire Line
+	3600 3200 2950 3200
+Wire Wire Line
+	2950 5250 3600 5250
+Wire Wire Line
 	2950 5450 3600 5450
 Wire Wire Line
-	2950 5250 3600 5250
-Wire Wire Line
-	3600 3200 2950 3200
-Wire Wire Line
-	2950 3000 3600 3000
-Wire Wire Line
-	2950 2800 3600 2800
-Wire Wire Line
-	3600 2100 2950 2100
-Wire Wire Line
-	2950 1700 3600 1700
-Wire Wire Line
-	6700 4400 5950 4400
-Wire Wire Line
-	5950 4400 5950 6950
-Wire Wire Line
-	5950 6950 10400 6950
-Wire Wire Line
-	10400 6950 10400 5000
-Wire Wire Line
-	10400 5000 10200 5000
-Wire Wire Line
-	10200 2500 10350 2500
-Wire Wire Line
-	10350 2500 10350 800
-Wire Wire Line
-	8200 4500 8800 4500
-Wire Wire Line
-	8200 4400 8800 4400
-Wire Wire Line
-	8200 4300 8800 4300
-Wire Wire Line
-	8200 4200 8800 4200
-Wire Wire Line
-	8200 6100 8350 6100
-Connection ~ 6150 4500
-Wire Wire Line
-	6150 2100 6150 5800
-Wire Wire Line
-	6150 5800 6700 5800
-Connection ~ 6350 4200
-Wire Wire Line
-	6350 5500 6350 1250
-Wire Wire Line
-	6350 5500 6700 5500
-Wire Wire Line
-	6700 6000 6550 6000
-Wire Wire Line
-	6550 6000 6550 5050
-Wire Wire Line
-	6550 5050 8550 5050
-Wire Wire Line
-	8550 5050 8550 4800
-Wire Wire Line
-	8550 4800 8200 4800
-Connection ~ 6050 3400
-Wire Wire Line
-	6700 4600 6050 4600
-Connection ~ 6450 3100
-Wire Wire Line
-	6450 4300 6700 4300
-Connection ~ 6250 4100
-Wire Wire Line
-	6250 4100 6700 4100
-Connection ~ 6050 2200
-Wire Wire Line
-	6050 3400 6700 3400
-Wire Wire Line
-	6450 3100 6700 3100
-Connection ~ 6250 2900
-Wire Wire Line
-	6250 2900 6700 2900
-Wire Wire Line
-	6700 3500 6550 3500
-Wire Wire Line
-	6550 3500 6550 2650
-Wire Wire Line
-	6550 2650 8500 2650
-Wire Wire Line
-	8500 2650 8500 2350
-Wire Wire Line
-	8500 2350 8200 2350
-Wire Wire Line
-	8800 3200 8200 3200
-Wire Wire Line
-	8800 3000 8200 3000
-Wire Wire Line
-	6700 2000 6150 2000
-Wire Wire Line
-	6150 2000 6150 800
-Wire Wire Line
-	6150 800  10350 800
-Wire Wire Line
-	5900 2550 5900 2500
-Wire Wire Line
-	5900 2550 8600 2550
-Wire Wire Line
-	8600 2550 8600 2250
-Wire Wire Line
-	8600 2250 8200 2250
-Connection ~ 6350 1800
-Wire Wire Line
-	6350 1250 8800 1250
-Connection ~ 6250 1700
-Wire Wire Line
-	6700 2100 5600 2100
-Wire Wire Line
-	6700 1800 5600 1800
-Wire Wire Line
-	6700 2300 5600 2300
-Wire Wire Line
-	8200 1800 8800 1800
-Wire Wire Line
-	8200 2000 8800 2000
-Wire Wire Line
-	8200 2100 8800 2100
-Wire Wire Line
-	8200 1900 8800 1900
-Wire Wire Line
-	5600 1700 6700 1700
-Wire Wire Line
-	5600 1900 6700 1900
-Wire Wire Line
-	5600 2200 6700 2200
-Wire Wire Line
-	8800 1150 6250 1150
-Wire Wire Line
-	8800 1350 6450 1350
-Connection ~ 6450 1900
-Wire Wire Line
-	5900 2500 5600 2500
-Wire Wire Line
-	8200 2900 8800 2900
-Wire Wire Line
-	8200 3100 8800 3100
-Wire Wire Line
-	8200 3450 8800 3450
-Wire Wire Line
-	6350 3000 6700 3000
-Wire Wire Line
-	6150 3300 6700 3300
-Connection ~ 6150 2100
-Wire Wire Line
-	6350 4200 6700 4200
-Connection ~ 6350 3000
-Wire Wire Line
-	6150 4500 6700 4500
-Connection ~ 6150 3300
-Wire Wire Line
-	8200 3550 8500 3550
-Wire Wire Line
-	8500 3550 8500 3750
-Wire Wire Line
-	8500 3750 6550 3750
-Wire Wire Line
-	6550 3750 6550 4700
-Wire Wire Line
-	6550 4700 6700 4700
-Wire Wire Line
-	6700 5400 6250 5400
-Wire Wire Line
-	6700 5600 6450 5600
-Wire Wire Line
-	6450 5600 6450 1350
-Connection ~ 6450 4300
-Wire Wire Line
-	6700 5900 6050 5900
-Wire Wire Line
-	6050 5900 6050 2200
-Connection ~ 6050 4600
-Wire Wire Line
-	6700 5700 6650 5700
-Wire Wire Line
-	6650 5700 6650 6400
-Wire Wire Line
-	8200 5500 8800 5500
-Wire Wire Line
-	8200 5600 8800 5600
-Wire Wire Line
-	8200 5700 8800 5700
-Wire Wire Line
-	8200 5800 8800 5800
-Wire Wire Line
-	8200 6000 8800 6000
-Wire Wire Line
-	8200 4700 8400 4700
-Wire Wire Line
-	8400 4700 8400 3850
-Wire Wire Line
-	8400 3850 6650 3850
-Wire Wire Line
-	6650 3850 6650 3200
-Wire Wire Line
-	6650 3200 6700 3200
-Wire Wire Line
-	6250 5400 6250 1150
-Wire Wire Line
-	3600 1900 2950 1900
-Wire Wire Line
-	2950 2200 3600 2200
-Wire Wire Line
-	3600 2900 2950 2900
-Wire Wire Line
-	3600 3100 2950 3100
-Wire Wire Line
-	3600 5150 2950 5150
-Wire Wire Line
-	3600 5350 2950 5350
+	2950 1800 3600 1800
 $Sheet
 S 1500 5000 1450 600
@@
 F29 "BTN2" I L 3600 4000 60
 F30 "BTN1" I L 3600 4100 60
-F31 "DAC" O L 3600 2400 60
-F32 "FLASH_CS" O L 3600 5450 60
-F33 "FLASH_SPI_SCK" O L 3600 5350 60
-F34 "FLASH_SPI_MOSI" O L 3600 5150 60
-F35 "FLASH_SPI_MISO" I L 3600 5250 60
+F31 "FLASH_CS" O L 3600 5450 60
+F32 "FLASH_SPI_SCK" O L 3600 5350 60
+F33 "FLASH_SPI_MOSI" O L 3600 5150 60
+F34 "FLASH_SPI_MISO" I L 3600 5250 60
+F35 "MIDI_RX2" I L 3600 2000 60
 $EndSheet
 $Sheet
@@
 F4 "USB_DM" B R 2950 2200 60
 F5 "USB_DP" B R 2950 2100 60
+F6 "MIDI_RX2" O R 2950 2000 60
+F7 "MIDI_TX2" I R 2950 1800 60
 $EndSheet
 $Sheet
@@
 $EndSheet
 $Comp
-L GND #PWR2
+L GND #PWR01
 U 1 1 4F8DA5D4
 P 6650 6400
-F 0 "#PWR2" H 6650 6400 30  0001 C CNN
+F 0 "#PWR01" H 6650 6400 30  0001 C CNN
 F 1 "GND" H 6650 6330 30  0001 C CNN
 	1    6650 6400

Commit message: Work.
Changed lines of the file:
@@
-EESchema Schematic File Version 2  date Sun 16 Dec 2012 05:53:49 PM CET
+EESchema Schematic File Version 2  date Sun 05 May 2013 06:02:32 PM CEST
 LIBS:power
 LIBS:device
@@
 Sheet 1 10
 Title ""
-Date "16 dec 2012"
+Date "5 may 2013"
 Rev ""
 Comp ""
@@
 $EndDescr
 Wire Wire Line
+	2950 5000 3600 5000
+Wire Wire Line
+	2950 4900 3600 4900
+Wire Wire Line
+	2950 4800 3600 4800
+Wire Wire Line
+	2950 4700 3600 4700
+Wire Wire Line
+	2950 4400 3600 4400
+Wire Wire Line
+	2950 4300 3600 4300
+Wire Wire Line
+	2950 4200 3600 4200
+Wire Wire Line
+	2950 4100 3600 4100
+Wire Wire Line
+	2950 4000 3600 4000
+Wire Wire Line
+	2950 3800 3600 3800
+Wire Wire Line
+	2950 3700 3600 3700
+Wire Wire Line
+	2950 3600 3600 3600
+Wire Wire Line
+	2950 3400 3600 3400
+Wire Wire Line
 	3600 2000 2950 2000
 Wire Wire Line
-	3600 5350 2950 5350
-Wire Wire Line
-	3600 5150 2950 5150
+	3600 5650 2950 5650
+Wire Wire Line
+	3600 5450 2950 5450
 Wire Wire Line
 	3600 3100 2950 3100
@@
 Connection ~ 6150 3300
 Wire Wire Line
-	6150 4500 6700 4500
+	6700 4500 6150 4500
 Connection ~ 6350 3000
 Wire Wire Line
@@
 	6250 1150 8800 1150
 Wire Wire Line
-	5600 2200 6700 2200
-Wire Wire Line
-	5600 1900 6700 1900
-Wire Wire Line
-	5600 1700 6700 1700
+	6700 2200 5600 2200
+Wire Wire Line
+	6700 1900 5600 1900
+Wire Wire Line
+	6700 1700 5600 1700
 Wire Wire Line
 	8200 1900 8800 1900
@@
 	6700 2300 5600 2300
 Wire Wire Line
-	6700 1800 5600 1800
-Wire Wire Line
-	6700 2100 5600 2100
+	5600 1800 6700 1800
+Wire Wire Line
+	5600 2100 6700 2100
 Connection ~ 6250 1700
 Wire Wire Line
@@
 	3600 3200 2950 3200
 Wire Wire Line
-	2950 5250 3600 5250
-Wire Wire Line
-	2950 5450 3600 5450
+	2950 5550 3600 5550
+Wire Wire Line
+	2950 5750 3600 5750
 Wire Wire Line
 	2950 1800 3600 1800
-$Sheet
-S 1500 5000 1450 600
+Wire Wire Line
+	3600 3500 2950 3500
+$Sheet
+S 1500 2700 1450 2400
+U 50CC7DE6
+F0 "panel" 60
+F1 "panel.sch" 60
+F2 "BACKLIGHT_PWM" I R 2950 2800 60
+F3 "LCD_SPI_MOSI" I R 2950 3200 60
+F4 "LCD_SPI_SCK" I R 2950 3100 60
+F5 "LCD_A0" I R 2950 3000 60
+F6 "LCD_CS" I R 2950 2900 60
+F7 "LED4" I R 2950 4700 60
+F8 "LED3" I R 2950 4800 60
+F9 "LED2" I R 2950 4900 60
+F10 "LED1" I R 2950 5000 60
+F11 "BTN5" O R 2950 4400 60
+F12 "BTN4" O R 2950 4300 60
+F13 "BTN3" O R 2950 4200 60
+F14 "BTN2" O R 2950 4100 60
+F15 "BTN1" O R 2950 4000 60
+F16 "ENCODER2" O R 2950 3400 60
+F17 "ENCODER1" O R 2950 3500 60
+F18 "ENC_BTN" O R 2950 3800 60
+F19 "ENC_LED2" I R 2950 3600 60
+F20 "ENC_LED1" I R 2950 3700 60
+$EndSheet
+$Sheet
+S 1500 5300 1450 600
 U 50CC8305
 F0 "flash" 60
 F1 "flash.sch" 60
-F2 "FLASH_SPI_MOSI" I R 2950 5150 60
-F3 "FLASH_SPI_SCK" I R 2950 5350 60
-F4 "FLASH_SPI_MISO" O R 2950 5250 60
-F5 "FLASH_CS" I R 2950 5450 60
+F2 "FLASH_SPI_MOSI" I R 2950 5450 60
+F3 "FLASH_SPI_SCK" I R 2950 5650 60
+F4 "FLASH_SPI_MISO" O R 2950 5550 60
+F5 "FLASH_CS" I R 2950 5750 60
 $EndSheet
 $Sheet
@@
 F19 "ENCODER2" I L 3600 3400 60
 F20 "ENCODER1" I L 3600 3500 60
-F21 "LED5" O L 3600 4300 60
-F22 "LED4" O L 3600 4400 60
-F23 "LED3" O L 3600 4500 60
-F24 "LED2" O L 3600 4600 60
-F25 "LED1" O L 3600 4700 60
-F26 "BTN5" I L 3600 3700 60
-F27 "BTN4" I L 3600 3800 60
-F28 "BTN3" I L 3600 3900 60
-F29 "BTN2" I L 3600 4000 60
-F30 "BTN1" I L 3600 4100 60
-F31 "FLASH_CS" O L 3600 5450 60
-F32 "FLASH_SPI_SCK" O L 3600 5350 60
-F33 "FLASH_SPI_MOSI" O L 3600 5150 60
-F34 "FLASH_SPI_MISO" I L 3600 5250 60
-F35 "MIDI_RX2" I L 3600 2000 60
+F21 "LED4" O L 3600 4700 60
+F22 "LED3" O L 3600 4800 60
+F23 "LED2" O L 3600 4900 60
+F24 "LED1" O L 3600 5000 60
+F25 "BTN5" I L 3600 4000 60
+F26 "BTN4" I L 3600 4100 60
+F27 "BTN3" I L 3600 4200 60
+F28 "BTN2" I L 3600 4300 60
+F29 "BTN1" I L 3600 4400 60
+F30 "FLASH_CS" O L 3600 5750 60
+F31 "FLASH_SPI_SCK" O L 3600 5650 60
+F32 "FLASH_SPI_MOSI" O L 3600 5450 60
+F33 "FLASH_SPI_MISO" I L 3600 5550 60
+F34 "MIDI_RX2" I L 3600 2000 60
+F35 "ENC_BTN" I L 3600 3800 60
+F36 "ENC_LED2" O L 3600 3600 60
+F37 "ENC_LED1" O L 3600 3700 60
 $EndSheet
 $Sheet
@@
 F6 "MIDI_RX2" O R 2950 2000 60
 F7 "MIDI_TX2" I R 2950 1800 60
-$EndSheet
-$Sheet
-S 1500 2700 1450 2100
-U 50CC7DE6
-F0 "panel" 60
-F1 "panel.sch" 60
-F2 "BACKLIGHT_PWM" I R 2950 2800 60
-F3 "LCD_SPI_MOSI" I R 2950 3200 60
-F4 "LCD_SPI_SCK" I R 2950 3100 60
-F5 "LCD_A0" I R 2950 3000 60
-F6 "LCD_CS" I R 2950 2900 60
-F7 "LED5" I R 2950 4300 60
-F8 "LED4" I R 2950 4400 60
-F9 "LED3" I R 2950 4500 60
-F10 "LED2" I R 2950 4600 60
-F11 "LED1" I R 2950 4700 60
-F12 "BTN5" O R 2950 3700 60
-F13 "BTN4" O R 2950 3800 60
-F14 "BTN3" O R 2950 3900 60
-F15 "BTN2" O R 2950 4000 60
-F16 "BTN1" O R 2950 4100 60
 $EndSheet
 NoConn ~ 8350 6100
@@
 $EndSheet
 $Comp
-L GND #PWR01
+L GND #PWR1
 U 1 1 4F8DA5D4
 P 6650 6400
-F 0 "#PWR01" H 6650 6400 30  0001 C CNN
+F 0 "#PWR1" H 6650 6400 30  0001 C CNN
 F 1 "GND" H 6650 6330 30  0001 C CNN
 	1    6650 6400

Commit message: Layouting.
Parts:
- added TP11: TST, symbol TST
Connections:
- net encoders/SHIFT_CLK: now also TP11.1

Commit message: Finished board CAD?
Parts:
- removed H10, H9: CONN_1, symbol CONN_1
Changed lines of the file:
@@
-EESchema Schematic File Version 2  date Sat 01 Jun 2013 11:43:44 AM CEST
+EESchema Schematic File Version 2  date Sat 08 Jun 2013 11:15:40 AM CEST
 LIBS:power
 LIBS:device
@@
 Sheet 1 10
 Title ""
-Date "1 jun 2013"
+Date "8 jun 2013"
 Rev ""
 Comp ""
@@
 F14 "SW1" O R 8200 4200 60
 $EndSheet
-$Comp
-L CONN_1 H10
-U 1 1 4F90F9F5
-P 3600 1000
-F 0 "H10" H 3680 1000 40  0000 L CNN
-F 1 "CONN_1" H 3600 1055 30  0001 C CNN
-	1    3600 1000
-	0    -1   -1   0
-$EndComp
-$Comp
-L CONN_1 H9
-U 1 1 4F90F9F3
-P 3500 1000
-F 0 "H9" H 3580 1000 40  0000 L CNN
-F 1 "CONN_1" H 3500 1055 30  0001 C CNN
-	1    3500 1000
-	0    -1   -1   0
-$EndComp
 Text Notes 3400 760  2    60   ~ 0
 Mounting holes
@@
 $EndSheet
 $Comp
-L GND #PWR1
+L GND #PWR01
 U 1 1 4F8DA5D4
 P 6650 6400
-F 0 "#PWR1" H 6650 6400 30  0001 C CNN
+F 0 "#PWR01" H 6650 6400 30  0001 C CNN
 F 1 "GND" H 6650 6330 30  0001 C CNN
 	1    6650 6400
