File: stm32.sch (KiCad schematic (older format))
At the start: 4 parts, among them U2 STM32F102CX

Commit message: updates.
Parts:
- added C1, C13, C14, C15, C4: C, symbol C
- added C12, C2: pF, symbol C
- added C18, C19, C20, C21, C22, C23, C24, C25: 1u, symbol C
- added C5: CP1, symbol CP1
- added LCD1: NHD-LCD, symbol NHD-LCD
- added P2: CONN_5X2, symbol CONN_5X2
- added Q1: BC237, TO92-EBC, symbol BC237
- added R1, R2, R3, R4: 10k, symbol R
- added R31, R32, R33, R34, R35, R36, R5: R, symbol R
- added R6: 100k, symbol R
- added SW1, SW2, SW3, SW4: SW_PUSH, symbol SW_PUSH
- added U1: SPI-FLASH, symbol SPI-FLASH
- added U6: LP2985LV, symbol LP2985LV
- added X1: CRYSTAL, symbol CRYSTAL
- gave numbers to parts that had none: 3
Connections:
- net labels added: +3.3V, BACK, BOOT0, BUF_OE1, BUF_OE2, BUF_OE3, BUF_OE4, BUF_OE5, BUF_OE6, BUS_0, BUS_1, BUS_2, BUS_3, BUS_4, BUS_5, BUS_6, BUS_7, CS_FLASH, CS_LCD, ENTER, GND, LCD_A0, LEFT, OSCIN, OSCOUT, PGM_RX, PGM_TX, RIGHT, RST, SWCLK, SWDIO, VPULLUP
- net labels removed: BOOTJUMPER, BTN_1, BTN_2, LED_OE
- wire segments 38 -> 153
- no-connect marks 0 -> 3
Other:
- note added: "Boot modes:\nBOOT1:BOOT0 = x0 --> flash\nBOOT1:BOOT0 = 01 --> bootloader"
- note added: "Boot pull-down."
- note added: "Cortex Debug"
- note added: "Find a suitable 3V3 regulator.\nWhat's our current demands?\nLEDs are on raw 5V.\nDecoupling demands?"
- note added: "Needs a resistor?"
- note added: "Needs current limiting\nresistor for LED?"
- note added: "Pullup current enough to drive\n* transistor for LCD backlight\n* 48 10k resistors to ground worst case (=15.84mA)\nConsider a transistor here, or weaker pullups."
- note added: "This display (NHD-C12832A1Z-FSW-FBW-3V3) isn't really SPI.\nCheck the data sheet for the controller (linked from the display\ndata sheet) to see if we've missed something."
- note added: "encoder output\nbuffer enables\n(active low)"
- note added: "what??"
- note removed: "Boot pull-down.\nWhat will the latch\nthink of this?"
- note removed: "Might need pullups\non these, depending\non what a dangling pin\non the chip does."
- note removed: "encoder\noutput\nlatch\nenables"
- moved on the sheet: C10, C9, R29

Commit message: Minor
Parts:
- added C7: 1u, symbol C
- added C8: 100n, symbol C
- added R7: DNP, symbol R
- added R8: 10k, symbol R
- added R9: R, symbol R
- C10: value CP1 -> 10u
- C13, C14, C15, C9: value C -> 100n
- R29, R31, R32, R33, R34, R35, R36, R5: value R -> 10k
Connections:
- wire segments 153 -> 162
Other:
- note added: "AN2586 recommends 100n on all power pins,\nplus one 10uF, plus another 1u on VDDA-VSSA.\nPlace small caps (at least 0805) for smaller impedance."
- note added: "Big decoupling for pgm current?"
- note added: "Find a suitable 3V3 regulator.\nWhat's our current demands?\nLEDs are on raw 5V.\nDecoupling demands? Big can on 5V for LEDs?"
- note added: "Needs current limiting resistor for LED?\nDiscreet NPN (is 10k small enough on the base)?\n...or a SOT23 NPN with built-in biasing."
- note added: "This display (NHD-C12832A1Z-FSW-FBW-3V3) isn't really SPI.\nCheck the data sheet for the controller (linked from the display\ndata sheet) to see if we've missed something.\nWhy is there only 16 pins on the module???"
- note added: "Want a small package (0805),\npossibly zero ohms."
- note added: "encoder output buffer\nenables (active low).\nPullup values are not critical,\nMCU can drive high after boot."
- note removed: "Find a suitable 3V3 regulator.\nWhat's our current demands?\nLEDs are on raw 5V.\nDecoupling demands?"
- note removed: "Needs a resistor?"
- note removed: "Needs current limiting\nresistor for LED?"
- note removed: "This display (NHD-C12832A1Z-FSW-FBW-3V3) isn't really SPI.\nCheck the data sheet for the controller (linked from the display\ndata sheet) to see if we've missed something."
- note removed: "encoder output\nbuffer enables\n(active low)"
- moved on the sheet: C1

Commit message: Updates
Parts:
- removed C4: C, symbol C
- removed C8: 100n, symbol C
- removed U6: LP2985LV, symbol LP2985LV
- added C17: 100u, symbol CP1
- added C4: 10u, symbol CP1
- added U6: LM1117, symbol LM1117
- C5: value CP1 -> 10u
Connections:
- net labels added: +5V
- wire segments 162 -> 174
Other:
- note added: "AN2586 recommends 100n on all power pins,\nplus one 10uF, plus another 1u on VDDA-VSSA.\nWe're ignoring the 100n on VDDA, because the 1u is in the\nsame package (0805) with the same impedance.\nPlace small caps (at least 0805) for smaller impedance."
- note added: "Find a suitable 3V3 regulator.\nWhat's our current demands?\nLEDs are on raw 5V.\nDecoupling demands? Big can on 5V for LEDs?\n\n100u 16V: UUR1C101MCL1GS (0.15€). φ8 × 6.2\n10u available in 1206 or 0805 @ 0.074€.\n100n available in 0805 @ 1.7€ for 100.\n\n771-NX1117C33Z115 is 0.2€, fixed 3.3V 1A, 1.2V dropout.\nSOT223, tab is VOUT. Wants 10u on in and out."
- note removed: "AN2586 recommends 100n on all power pins,\nplus one 10uF, plus another 1u on VDDA-VSSA.\nPlace small caps (at least 0805) for smaller impedance."
- note removed: "Find a suitable 3V3 regulator.\nWhat's our current demands?\nLEDs are on raw 5V.\nDecoupling demands? Big can on 5V for LEDs?"
- moved on the sheet: C5
