File: stm32.sch (KiCad schematic (older format))
At the start: 47 parts, among them P2 CONN_5X2, Q1 BC237, SW1 SW_PUSH, SW2 SW_PUSH, SW3 SW_PUSH, SW4 SW_PUSH, U1 SPI-FLASH, U2 STM32F102CX, U6 LM1117, X1 CRYSTAL

Commit message: Display and crystal.
Parts:
- removed C18, C19, C20, C21, C22, C23, C24, C25: 1u, symbol C
- removed LCD1: NHD-LCD, symbol NHD-LCD
- added LCD2: DOGS102-6, symbol DOGS102-6
- X1: value CRYSTAL -> 8MHz
Connections:
- wire segments 174 -> 151
Other:
- note added: "ABLS-8.000MHZ-B2-T\nHC-49/US"
- moved on the sheet: R8

Commit message: Package updates
Parts:
- removed C10: 10u, symbol CP1
- removed Q1: BC237, TO92-EBC, symbol BC237
- removed R8: 10k, symbol R
- added C10: 10u, symbol C
- added C18, C19, C20: 1u, symbol C
- added C21: DNP, symbol C
- added C8: 100n, symbol C
- added Q3: PDTC123Y, SOT23-3, symbol PDTC123Y
- added R11: 35, symbol R
- C1: value C -> 100n
- R29, R31, R32, R33, R34, R35, R36, R5: value 10k -> 20k
- U1: value SPI-FLASH -> AT25DF081A-SH
Connections:
- wire segments 151 -> 182
Other:
- note added: "Backlight at 5V, 80mA, Vf=2.2V --> 35ohm (0.25W),\nignoring drop in transistor. Base resistor\ncould be about 5k."
- note added: "Decoupling demands? Big can on 5V for LEDs?\n100u 16V: UUR1C101MCL1GS (0.15€). φ8 × 6.2\n10u available in 1206 or 0805 @ 0.074€.\n100n available in 0805 @ 1.7€ for 100.\n\n771-NX1117C33Z115 is 0.2€, fixed 3.3V 1A, 1.2V dropout.\nSOT223, tab is VOUT. Wants 10u on in and out."
- note removed: "Big decoupling for pgm current?"
- note removed: "Find a suitable 3V3 regulator.\nWhat's our current demands?\nLEDs are on raw 5V.\nDecoupling demands? Big can on 5V for LEDs?\n\n100u 16V: UUR1C101MCL1GS (0.15€). φ8 × 6.2\n10u available in 1206 or 0805 @ 0.074€.\n100n available in 0805 @ 1.7€ for 100.\n\n771-NX1117C33Z115 is 0.2€, fixed 3.3V 1A, 1.2V dropout.\nSOT223, tab is VOUT. Wants 10u on in and out."
- note removed: "Needs current limiting resistor for LED?\nDiscreet NPN (is 10k small enough on the base)?\n...or a SOT23 NPN with built-in biasing."
- moved on the sheet: C1, U1

Commit message: Changes.
Parts:
- removed SW1, SW2, SW3, SW4: SW_PUSH, symbol SW_PUSH
- added SW1, SW2, SW3, SW4: 101-0661-EV, symbol TACT
- R1, R2, R3, R4: value 10k -> 20k

Commit message: Floorplanning
Parts:
- added C22: 100n, symbol C
Connections:
- wire segments 182 -> 184
Changed lines of the file:
@@
-EESchema Schematic File Version 2  date Sat 14 Apr 2012 07:12:50 PM CEST
+EESchema Schematic File Version 2  date Sun 15 Apr 2012 10:50:25 AM CEST
 LIBS:power
 LIBS:device
@@
 Sheet 4 5
 Title ""
-Date "14 apr 2012"
+Date "15 apr 2012"
 Rev ""
 Comp ""
@@
 Comment4 ""
 $EndDescr
+Wire Wire Line
+	9150 2250 8900 2250
 Connection ~ 2850 1700
 Wire Wire Line
@@
 	10950 4000 10950 3950
 Wire Wire Line
-	8900 1850 8900 1800
+	8900 1800 8900 1850
 Wire Wire Line
 	9700 1600 9700 1700
@@
 	9700 1150 9700 1200
 Wire Wire Line
-	8900 2300 8900 2250
+	8900 2250 8900 2300
 Wire Wire Line
 	10950 3550 10950 3500
@@
 	3600 2000 2850 2000
 Connection ~ 2850 2000
+Wire Wire Line
+	8900 1850 9150 1850
+$Comp
+L C C22
+U 1 1 4F8A80A9
+P 9150 2050
+F 0 "C22" H 9200 2150 50  0000 L CNN
+F 1 "100n" H 9200 1950 50  0000 L CNN
+	1    9150 2050
+	1    0    0    -1
+$EndComp
 $Comp
 L TACT SW4

Commit message: Switch to shift registers. Routing.
Parts:
- removed R31, R32, R33, R34, R35, R36: 20k, symbol R
Connections:
- net labels added: BOOT1, BTN1, BTN2, BTN3, BTN4, BTN_CE, BTN_LOAD, BTN_SHIFT, JTDI, JTDO, LED_LOAD, LED_OE, LED_SHIFT, SHIFT_CLK
- net labels removed: BACK, BUF_OE1, BUF_OE2, BUF_OE3, BUF_OE4, BUF_OE5, BUF_OE6, BUS_0, BUS_1, BUS_2, BUS_3, BUS_4, BUS_5, BUS_6, BUS_7, ENTER, LED_CLK, LED_DATA, LED_LATCH, LEFT, RIGHT
- wire segments 184 -> 160
- no-connect marks 3 -> 9
Other:
- note removed: "encoder output buffer\nenables (active low).\nPullup values are not critical,\nMCU can drive high after boot."
- note removed: "encoder\noutputs\nthrough\nbuffers/latches"
- note removed: "what??"
- moved on the sheet: R29, R7
