File: stm32.sch (KiCad schematic (older format))
At the start: 15 parts, among them U6 LM1117, X1 8MHz

Commit message: Chaotic changes.
Parts:
- removed P?: CONN_10X2, symbol CONN_10X2
- added C33: 100n, symbol C
- added P2: CONN_5X2, symbol CONN_5X2
- added TP0, TP10, TP11, TP9: TST, symbol TST
- gave numbers to parts that had none: 1
Connections:
- net labels added: MIDI_RX2, SWO
- net labels removed: DAC
- wire segments 47 -> 88
- no-connect marks 0 -> 2
Other:
- note added: "Add test points on SPI busses, shift regs, some unused pins."
- note removed: "Pullup current enough to drive\n* 48 10k resistors to ground worst case (=15.84mA)\nConsider a transistor here, or weaker pullups."

Commit message: Work.
Connections:
- net ENC_BTN: now reaches U2.14 (PA0-WKUP)
- net ENC_LED2: now reaches U2.51 (PC10)
- net LED5 renamed ENC_LED1

Commit message: Routing.
Parts:
- removed TP11: TST, symbol TST
- added TP12: TST, symbol TST
Connections:
- net GND: now also TP12.1
Changed lines of the file:
@@
-EESchema Schematic File Version 2  date Sun 05 May 2013 06:02:32 PM CEST
+EESchema Schematic File Version 2  date Wed 08 May 2013 08:54:31 PM CEST
 LIBS:power
 LIBS:device
@@
 Sheet 4 10
 Title ""
-Date "5 may 2013"
+Date "8 may 2013"
 Rev ""
 Comp ""
@@
 Comment4 ""
 $EndDescr
+$Comp
+L TST TP12
+U 1 1 5189413B
+P 6600 6000
+F 0 "TP12" H 6600 6300 40  0000 C CNN
+F 1 "TST" H 6600 6250 30  0000 C CNN
+	1    6600 6000
+	0    1    1    0
+$EndComp
 Wire Wire Line
 	3050 3700 3200 3700
@@
 Add test points on SPI busses, shift regs, some unused pins.
 $Comp
-L TST TP11
-U 1 1 50CDE40E
-P 9000 3800
-F 0 "TP11" H 9000 4100 40  0000 C CNN
-F 1 "TST" H 9000 4050 30  0000 C CNN
-	1    9000 3800
-	1    0    0    -1
-$EndComp
-$Comp
 L TST TP0
 U 1 1 50CDE3D7
@@
 MIDI_RX2
 $Comp
-L GND #PWR36
+L GND #PWR022
 U 1 1 50CDD646
 P 9200 2100
-F 0 "#PWR36" H 9200 2100 30  0001 C CNN
+F 0 "#PWR022" H 9200 2100 30  0001 C CNN
 F 1 "GND" H 9200 2030 30  0001 C CNN
 	1    9200 2100
@@
 NoConn ~ 10150 2000
 $Comp
-L +3.3V #PWR33
+L +3.3V #PWR023
 U 1 1 50CDD48A
 P 9200 1700
-F 0 "#PWR33" H 9200 1660 30  0001 C CNN
+F 0 "#PWR023" H 9200 1660 30  0001 C CNN
 F 1 "+3.3V" H 9200 1810 30  0000 C CNN
 	1    9200 1700
@@
 $EndComp
 $Comp
-L GND #PWR35
+L GND #PWR024
 U 1 1 50CDD483
 P 9200 1900
-F 0 "#PWR35" H 9200 1900 30  0001 C CNN
+F 0 "#PWR024" H 9200 1900 30  0001 C CNN
 F 1 "GND" H 9200 1830 30  0001 C CNN
 	1    9200 1900
@@
 $EndComp
 $Comp
-L GND #PWR34
+L GND #PWR025
 U 1 1 50CDD47F
 P 9200 1800
-F 0 "#PWR34" H 9200 1800 30  0001 C CNN
+F 0 "#PWR025" H 9200 1800 30  0001 C CNN
 F 1 "GND" H 9200 1730 30  0001 C CNN
 	1    9200 1800
@@
 $EndComp
 $Comp
-L GND #PWR39
+L GND #PWR026
 U 1 1 50CC9E8D
 P 10700 2600
-F 0 "#PWR39" H 10700 2600 30  0001 C CNN
+F 0 "#PWR026" H 10700 2600 30  0001 C CNN
 F 1 "GND" H 10700 2530 30  0001 C CNN
 	1    10700 2600
@@
 BTN1
 $Comp
-L GND #PWR29
+L GND #PWR027
 U 1 1 50CC7C9F
 P 6400 4100
-F 0 "#PWR29" H 6400 4100 30  0001 C CNN
+F 0 "#PWR027" H 6400 4100 30  0001 C CNN
 F 1 "GND" H 6400 4030 30  0001 C CNN
 	1    6400 4100
@@
 RST
 $Comp
-L GND #PWR28
+L GND #PWR028
 U 1 1 50CC762B
 P 6350 3300
-F 0 "#PWR28" H 6350 3300 30  0001 C CNN
+F 0 "#PWR028" H 6350 3300 30  0001 C CNN
 F 1 "GND" H 6350 3230 30  0001 C CNN
 	1    6350 3300
@@
 ABLS-8.000MHZ-B2-T\nHC-49/US\nESR max 80ohm
 $Comp
-L +5V #PWR32
+L +5V #PWR029
 U 1 1 4F834C8B
 P 8900 6200
-F 0 "#PWR32" H 8900 6290 20  0001 C CNN
+F 0 "#PWR029" H 8900 6290 20  0001 C CNN
 F 1 "+5V" H 8900 6290 30  0000 C CNN
 	1    8900 6200
@@
 $EndComp
 $Comp
-L GND #PWR37
+L GND #PWR030
 U 1 1 4F832167
 P 9650 7000
-F 0 "#PWR37" H 9650 7000 30  0001 C CNN
+F 0 "#PWR030" H 9650 7000 30  0001 C CNN
 F 1 "GND" H 9650 6930 30  0001 C CNN
 	1    9650 7000
@@
 $EndComp
 $Comp
-L GND #PWR24
+L GND #PWR031
 U 1 1 4F8288D9
 P 2600 6150
-F 0 "#PWR24" H 2600 6150 30  0001 C CNN
+F 0 "#PWR031" H 2600 6150 30  0001 C CNN
 F 1 "GND" H 2600 6080 30  0001 C CNN
 	1    2600 6150
@@
 $EndComp
 $Comp
-L +3.3V #PWR38
+L +3.3V #PWR032
 U 1 1 4F805934
 P 10450 6100
-F 0 "#PWR38" H 10450 6060 30  0001 C CNN
+F 0 "#PWR032" H 10450 6060 30  0001 C CNN
 F 1 "+3.3V" H 10450 6210 30  0000 C CNN
 	1    10450 6100
@@
 Boot modes:\nBOOT1:BOOT0 = x0 --> flash\nBOOT1:BOOT0 = 01 --> bootloader
 $Comp
-L +3.3V #PWR26
+L +3.3V #PWR033
 U 1 1 4F804819
 P 3650 7100
-F 0 "#PWR26" H 3650 7060 30  0001 C CNN
+F 0 "#PWR033" H 3650 7060 30  0001 C CNN
 F 1 "+3.3V" H 3650 7210 30  0000 C CNN
 	1    3650 7100
@@
 $EndComp
 $Comp
-L GND #PWR27
+L GND #PWR034
 U 1 1 4F804810
 P 3650 7650
-F 0 "#PWR27" H 3650 7650 30  0001 C CNN
+F 0 "#PWR034" H 3650 7650 30  0001 C CNN
 F 1 "GND" H 3650 7580 30  0001 C CNN
 	1    3650 7650
@@
 OSCIN
 $Comp
-L GND #PWR31
+L GND #PWR035
 U 1 1 4F804740
 P 7800 2650
-F 0 "#PWR31" H 7800 2650 30  0001 C CNN
+F 0 "#PWR035" H 7800 2650 30  0001 C CNN
 F 1 "GND" H 7800 2580 30  0001 C CNN
 	1    7800 2650
@@
 USB_DM
 $Comp
-L +3.3V #PWR25
+L +3.3V #PWR036
 U 1 1 4F802EBD
 P 2950 5350
-F 0 "#PWR25" H 2950 5310 30  0001 C CNN
+F 0 "#PWR036" H 2950 5310 30  0001 C CNN
 F 1 "+3.3V" H 2950 5460 30  0000 C CNN
 	1    2950 5350
@@
 $EndComp
 $Comp
-L GND #PWR30
+L GND #PWR037
 U 1 1 4F802EA6
 P 6600 6200
-F 0 "#PWR30" H 6600 6200 30  0001 C CNN
+F 0 "#PWR037" H 6600 6200 30  0001 C CNN
 F 1 "GND" H 6600 6130 30  0001 C CNN
 	1    6600 6200

Commit message: Layouting.
Parts:
- added TP14, TP15, TP16, TP17: TST, symbol TST
Connections:
- net at U2.15 (PA1): now also TP16.1
- net PA4: now reaches TP9.1, U2.20 (PA4)
- net at U2.52 (PC11): now also TP14.1
- net at U2.53 (PC12): now also TP15.1
- net at U2.54 (PD2): now also TP17.1

Commit message: Finished board layout.
Parts:
- added TP18, TP19: TST, symbol TST
Connections:
- net GND: now also TP0.1, TP18.1, TP19.1
Changed lines of the file:
@@
-EESchema Schematic File Version 2  date Sun 26 May 2013 03:42:57 PM CEST
+EESchema Schematic File Version 2  date Sat 01 Jun 2013 11:43:44 AM CEST
 LIBS:power
 LIBS:device
@@
 Sheet 4 10
 Title ""
-Date "26 may 2013"
+Date "1 jun 2013"
 Rev ""
 Comp ""
@@
 Comment4 ""
 $EndDescr
+Connection ~ 6600 5600
+Connection ~ 6600 5600
+$Comp
+L TST TP19
+U 1 1 51A9BDFC
+P 6600 5600
+F 0 "TP19" H 6600 5900 40  0000 C CNN
+F 1 "TST" H 6600 5850 30  0000 C CNN
+	1    6600 5600
+	0    1    1    0
+$EndComp
+$Comp
+L TST TP18
+U 1 1 51A9BCCE
+P 6600 5800
+F 0 "TP18" H 6600 6100 40  0000 C CNN
+F 1 "TST" H 6600 6050 30  0000 C CNN
+	1    6600 5800
+	0    1    1    0
+$EndComp
+Connection ~ 10200 6900
+Connection ~ 10200 6900
 Wire Wire Line
 	6400 3700 6200 3700
@@
 MIDI_RX2
 $Comp
-L GND #PWR021
+L GND #PWR33
 U 1 1 50CDD646
 P 9200 2100
-F 0 "#PWR021" H 9200 2100 30  0001 C CNN
+F 0 "#PWR33" H 9200 2100 30  0001 C CNN
 F 1 "GND" H 9200 2030 30  0001 C CNN
 	1    9200 2100
@@
 NoConn ~ 10150 2000
 $Comp
-L +3.3V #PWR022
+L +3.3V #PWR30
 U 1 1 50CDD48A
 P 9200 1700
-F 0 "#PWR022" H 9200 1660 30  0001 C CNN
+F 0 "#PWR30" H 9200 1660 30  0001 C CNN
 F 1 "+3.3V" H 9200 1810 30  0000 C CNN
 	1    9200 1700
@@
 $EndComp
 $Comp
-L GND #PWR023
+L GND #PWR32
 U 1 1 50CDD483
 P 9200 1900
-F 0 "#PWR023" H 9200 1900 30  0001 C CNN
+F 0 "#PWR32" H 9200 1900 30  0001 C CNN
 F 1 "GND" H 9200 1830 30  0001 C CNN
 	1    9200 1900
@@
 $EndComp
 $Comp
-L GND #PWR024
+L GND #PWR31
 U 1 1 50CDD47F
 P 9200 1800
-F 0 "#PWR024" H 9200 1800 30  0001 C CNN
+F 0 "#PWR31" H 9200 1800 30  0001 C CNN
 F 1 "GND" H 9200 1730 30  0001 C CNN
 	1    9200 1800
@@
 $EndComp
 $Comp
-L GND #PWR025
+L GND #PWR36
 U 1 1 50CC9E8D
 P 10700 2600
-F 0 "#PWR025" H 10700 2600 30  0001 C CNN
+F 0 "#PWR36" H 10700 2600 30  0001 C CNN
 F 1 "GND" H 10700 2530 30  0001 C CNN
 	1    10700 2600
@@
 BTN1
 $Comp
-L GND #PWR026
+L GND #PWR26
 U 1 1 50CC7C9F
 P 6400 4100
-F 0 "#PWR026" H 6400 4100 30  0001 C CNN
+F 0 "#PWR26" H 6400 4100 30  0001 C CNN
 F 1 "GND" H 6400 4030 30  0001 C CNN
 	1    6400 4100
@@
 RST
 $Comp
-L GND #PWR027
+L GND #PWR25
 U 1 1 50CC762B
 P 6350 3300
-F 0 "#PWR027" H 6350 3300 30  0001 C CNN
+F 0 "#PWR25" H 6350 3300 30  0001 C CNN
 F 1 "GND" H 6350 3230 30  0001 C CNN
 	1    6350 3300
@@
 ABLS-8.000MHZ-B2-T\nHC-49/US\nESR max 80ohm
 $Comp
-L +5V #PWR028
+L +5V #PWR29
 U 1 1 4F834C8B
 P 8900 6200
-F 0 "#PWR028" H 8900 6290 20  0001 C CNN
+F 0 "#PWR29" H 8900 6290 20  0001 C CNN
 F 1 "+5V" H 8900 6290 30  0000 C CNN
 	1    8900 6200
@@
 $EndComp
 $Comp
-L GND #PWR029
+L GND #PWR34
 U 1 1 4F832167
 P 9650 7000
-F 0 "#PWR029" H 9650 7000 30  0001 C CNN
+F 0 "#PWR34" H 9650 7000 30  0001 C CNN
 F 1 "GND" H 9650 6930 30  0001 C CNN
 	1    9650 7000
@@
 $EndComp
 $Comp
-L GND #PWR030
+L GND #PWR21
 U 1 1 4F8288D9
 P 2600 6150
-F 0 "#PWR030" H 2600 6150 30  0001 C CNN
+F 0 "#PWR21" H 2600 6150 30  0001 C CNN
 F 1 "GND" H 2600 6080 30  0001 C CNN
 	1    2600 6150
@@
 $EndComp
 $Comp
-L +3.3V #PWR031
+L +3.3V #PWR35
 U 1 1 4F805934
 P 10450 6100
-F 0 "#PWR031" H 10450 6060 30  0001 C CNN
+F 0 "#PWR35" H 10450 6060 30  0001 C CNN
 F 1 "+3.3V" H 10450 6210 30  0000 C CNN
 	1    10450 6100
@@
 Boot modes:\nBOOT1:BOOT0 = x0 --> flash\nBOOT1:BOOT0 = 01 --> bootloader
 $Comp
-L +3.3V #PWR032
+L +3.3V #PWR23
 U 1 1 4F804819
 P 3650 7100
-F 0 "#PWR032" H 3650 7060 30  0001 C CNN
+F 0 "#PWR23" H 3650 7060 30  0001 C CNN
 F 1 "+3.3V" H 3650 7210 30  0000 C CNN
 	1    3650 7100
@@
 $EndComp
 $Comp
-L GND #PWR033
+L GND #PWR24
 U 1 1 4F804810
 P 3650 7650
-F 0 "#PWR033" H 3650 7650 30  0001 C CNN
+F 0 "#PWR24" H 3650 7650 30  0001 C CNN
 F 1 "GND" H 3650 7580 30  0001 C CNN
 	1    3650 7650
@@
 OSCIN
 $Comp
-L GND #PWR034
+L GND #PWR28
 U 1 1 4F804740
 P 7800 2650
-F 0 "#PWR034" H 7800 2650 30  0001 C CNN
+F 0 "#PWR28" H 7800 2650 30  0001 C CNN
 F 1 "GND" H 7800 2580 30  0001 C CNN
 	1    7800 2650
@@
 USB_DM
 $Comp
-L +3.3V #PWR035
+L +3.3V #PWR22
 U 1 1 4F802EBD
 P 2950 5350
-F 0 "#PWR035" H 2950 5310 30  0001 C CNN
+F 0 "#PWR22" H 2950 5310 30  0001 C CNN
 F 1 "+3.3V" H 2950 5460 30  0000 C CNN
 	1    2950 5350
@@
 $EndComp
 $Comp
-L GND #PWR036
+L GND #PWR27
 U 1 1 4F802EA6
 P 6600 6200
-F 0 "#PWR036" H 6600 6200 30  0001 C CNN
+F 0 "#PWR27" H 6600 6200 30  0001 C CNN
 F 1 "GND" H 6600 6130 30  0001 C CNN
 	1    6600 6200

Commit message: Finished board CAD?
Parts:
- added D10, D9: LED, symbol LED
- added R29, R30: 390, symbol R
- C12, C2: value 16pF -> 15p
Connections:
- net GND: now also R29.2, R30.2
- net PA4: now also D10.1 (A)
- net PA1: now reaches TP16.1, U2.15 (PA1)
- net PA1: now also D9.1 (A)
- new net: D10.2 (K), R30.1
- new net: D9.2 (K), R29.1
Other:
- moved on the sheet: TP16, TP9
