File: switchbus.sch (KiCad schematic (older format))
At the start: 2 parts, among them U4 74HC245

Commit message: Package updates
Parts:
- C3: value C -> 100n
Changed lines of the file:
@@
-EESchema Schematic File Version 2  date Tue 10 Apr 2012 10:33:33 PM CEST
+EESchema Schematic File Version 2  date Sat 14 Apr 2012 04:28:33 PM CEST
 LIBS:power
 LIBS:device
@@
 LIBS:74hc
 LIBS:dogs102-6
+LIBS:pdt-transistor
 LIBS:knobboard-cache
 EELAYER 25  0
@@
 Sheet 2 5
 Title ""
-Date "10 apr 2012"
+Date "14 apr 2012"
 Rev ""
 Comp ""
@@
 P 4250 2600
 F 0 "C3" H 4300 2700 50  0000 L CNN
-F 1 "C" H 4300 2500 50  0000 L CNN
+F 1 "100n" H 4300 2500 50  0000 L CNN
 	1    4250 2600
 	1    0    0    -1

Commit message: Switch to shift registers. Routing.
Parts:
- removed U4: 74HC245, symbol 74LS245
- added U4: 74HC165, symbol 74LS165
Connections:
- net labels added: BTNSHIFT_IN0, BTNSHIFT_OUT0, BTN_CE, BTN_LOAD, SHIFT_CLK
- net labels removed: BUS_0, BUS_1, BUS_2, BUS_3, BUS_4, BUS_5, BUS_6, BUS_7, OE1
- wire segments 23 -> 8
- no-connect marks 0 -> 1
Other:
- moved on the sheet: C3
Changed lines of the file:
@@
-EESchema Schematic File Version 2  date Sun 15 Apr 2012 10:50:25 AM CEST
+EESchema Schematic File Version 2  date Tue 17 Apr 2012 08:42:54 PM CEST
 LIBS:power
 LIBS:device
@@
 Sheet 2 5
 Title ""
-Date "15 apr 2012"
+Date "17 apr 2012"
 Rev ""
 Comp ""
@@
 Comment4 ""
 $EndDescr
+NoConn ~ 4300 3000
 Wire Wire Line
-	4250 2800 4250 3000
+	2900 2800 2550 2800
 Wire Wire Line
-	6350 2050 6350 2200
+	5150 3100 5150 3250
 Wire Wire Line
-	5550 3100 5550 3150
+	5150 3650 5150 3850
 Wire Wire Line
-	5550 3150 5650 3150
+	2650 4000 2900 4000
 Wire Wire Line
-	7050 2950 7600 2950
+	2650 3750 2900 3750
 Wire Wire Line
-	7050 2850 7600 2850
+	3300 4050 3300 4250
 Wire Wire Line
-	7050 2750 7600 2750
+	3300 2500 3300 2750
 Wire Wire Line
-	7050 2650 7600 2650
-Wire Wire Line
-	7050 2550 7600 2550
-Wire Wire Line
-	7050 2450 7600 2450
-Wire Wire Line
-	7050 2350 7600 2350
-Wire Wire Line
-	7050 2250 7600 2250
-Wire Wire Line
-	5150 2250 5650 2250
-Wire Wire Line
-	5150 2350 5650 2350
-Wire Wire Line
-	5150 2450 5650 2450
-Wire Wire Line
-	5150 2550 5650 2550
-Wire Wire Line
-	5150 2650 5650 2650
-Wire Wire Line
-	5150 2750 5650 2750
-Wire Wire Line
-	5150 2850 5650 2850
-Wire Wire Line
-	5150 2950 5650 2950
-Wire Wire Line
-	5150 3250 5650 3250
-Wire Wire Line
-	6350 3300 6350 3450
-Wire Wire Line
-	4250 2250 4250 2400
+	2900 3900 2650 3900
 $Comp
-L GND #PWR01
-U 1 1 4F82A012
-P 4250 3000
-F 0 "#PWR01" H 4250 3000 30  0001 C CNN
-F 1 "GND" H 4250 2930 30  0001 C CNN
-	1    4250 3000
+L 74LS165 U4
+U 1 1 4F8DA66D
+P 3600 3400
+F 0 "U4" H 3750 3350 60  0000 C CNN
+F 1 "74HC165" H 3750 3150 60  0000 C CNN
+	1    3600 3400
 	1    0    0    -1
 $EndComp
 $Comp
-L +3.3V #PWR02
+L GND #PWR03
+U 1 1 4F8DA672
+P 3300 4250
+F 0 "#PWR03" H 3300 4250 30  0001 C CNN
+F 1 "GND" H 3300 4180 30  0001 C CNN
+	1    3300 4250
+	1    0    0    -1
+$EndComp
+$Comp
+L +3.3V #PWR04
+U 1 1 4F8DA671
+P 3300 2500
+F 0 "#PWR04" H 3300 2460 30  0001 C CNN
+F 1 "+3.3V" H 3300 2610 30  0000 C CNN
+	1    3300 2500
+	1    0    0    -1
+$EndComp
+Text HLabel 4300 2900 2    60   Output ~ 0
+BTNSHIFT_OUT0
+Text HLabel 2650 4000 0    60   Input ~ 0
+BTN_CE
+Text HLabel 2650 3750 0    60   Input ~ 0
+BTN_LOAD
+Text HLabel 2650 3900 0    60   Input ~ 0
+SHIFT_CLK
+Text HLabel 2550 2800 0    60   Input ~ 0
+BTNSHIFT_IN0
+$Comp
+L GND #PWR05
+U 1 1 4F82A012
+P 5150 3850
+F 0 "#PWR05" H 5150 3850 30  0001 C CNN
+F 1 "GND" H 5150 3780 30  0001 C CNN
+	1    5150 3850
+	1    0    0    -1
+$EndComp
+$Comp
+L +3.3V #PWR06
 U 1 1 4F82A00E
-P 4250 2250
-F 0 "#PWR02" H 4250 2210 30  0001 C CNN
-F 1 "+3.3V" H 4250 2360 30  0000 C CNN
-	1    4250 2250
+P 5150 3100
+F 0 "#PWR06" H 5150 3060 30  0001 C CNN
+F 1 "+3.3V" H 5150 3210 30  0000 C CNN
+	1    5150 3100
 	1    0    0    -1
 $EndComp
@@
 L C C3
 U 1 1 4F81BBEC
-P 4250 2600
-F 0 "C3" H 4300 2700 50  0000 L CNN
-F 1 "100n" H 4300 2500 50  0000 L CNN
-	1    4250 2600
+P 5150 3450
+F 0 "C3" H 5200 3550 50  0000 L CNN
+F 1 "100n" H 5200 3350 50  0000 L CNN
+	1    5150 3450
 	1    0    0    -1
 $EndComp
-Text HLabel 5150 3250 0    60   Input ~ 0
-OE1
-$Comp
-L GND #PWR03
-U 1 1 4F81A943
-P 6350 3450
-F 0 "#PWR03" H 6350 3450 30  0001 C CNN
-F 1 "GND" H 6350 3380 30  0001 C CNN
-	1    6350 3450
-	1    0    0    -1
-$EndComp
-$Comp
-L +3.3V #PWR04
-U 1 1 4F81A93C
-P 5550 3100
-F 0 "#PWR04" H 5550 3060 30  0001 C CNN
-F 1 "+3.3V" H 5550 3210 30  0000 C CNN
-	1    5550 3100
-	1    0    0    -1
-$EndComp
-$Comp
-L +3.3V #PWR05
-U 1 1 4F81A937
-P 6350 2050
-F 0 "#PWR05" H 6350 2010 30  0001 C CNN
-F 1 "+3.3V" H 6350 2160 30  0000 C CNN
-	1    6350 2050
-	1    0    0    -1
-$EndComp
-Text GLabel 7600 2950 2    60   BiDi ~ 0
-BUS_7
-Text GLabel 7600 2850 2    60   BiDi ~ 0
-BUS_6
-Text GLabel 7600 2750 2    60   BiDi ~ 0
-BUS_5
-Text GLabel 7600 2650 2    60   BiDi ~ 0
-BUS_4
-Text GLabel 7600 2550 2    60   BiDi ~ 0
-BUS_3
-Text GLabel 7600 2450 2    60   BiDi ~ 0
-BUS_2
-Text GLabel 7600 2350 2    60   BiDi ~ 0
-BUS_1
-Text GLabel 7600 2250 2    60   BiDi ~ 0
-BUS_0
-Text HLabel 5150 4350 0    60   Input ~ 0
+Text HLabel 7200 3850 0    60   Input ~ 0
 SW16
-Text HLabel 5150 4250 0    60   Input ~ 0
+Text HLabel 7200 3750 0    60   Input ~ 0
 SW15
-Text HLabel 5150 4150 0    60   Input ~ 0
+Text HLabel 7200 3650 0    60   Input ~ 0
 SW14
-Text HLabel 5150 4050 0    60   Input ~ 0
+Text HLabel 7200 3550 0    60   Input ~ 0
 SW13
-Text HLabel 5150 3950 0    60   Input ~ 0
+Text HLabel 7200 3450 0    60   Input ~ 0
 SW12
-Text HLabel 5150 3850 0    60   Input ~ 0
+Text HLabel 7200 3350 0    60   Input ~ 0
 SW11
-Text HLabel 5150 3750 0    60   Input ~ 0
+Text HLabel 7200 3250 0    60   Input ~ 0
 SW10
-Text HLabel 5150 3650 0    60   Input ~ 0
+Text HLabel 7200 3150 0    60   Input ~ 0
 SW9
-Text HLabel 5150 2950 0    60   Input ~ 0
+Text HLabel 2900 3600 0    60   Input ~ 0
 SW8
-Text HLabel 5150 2850 0    60   Input ~ 0
+Text HLabel 2900 3500 0    60   Input ~ 0
 SW7
-Text HLabel 5150 2750 0    60   Input ~ 0
+Text HLabel 2900 3400 0    60   Input ~ 0
 SW6
-Text HLabel 5150 2650 0    60   Input ~ 0
+Text HLabel 2900 3300 0    60   Input ~ 0
 SW5
-Text HLabel 5150 2550 0    60   Input ~ 0
+Text HLabel 2900 3200 0    60   Input ~ 0
 SW4
-Text HLabel 5150 2450 0    60   Input ~ 0
+Text HLabel 2900 3100 0    60   Input ~ 0
 SW3
-Text HLabel 5150 2350 0    60   Input ~ 0
+Text HLabel 2900 3000 0    60   Input ~ 0
 SW2
-Text HLabel 5150 2250 0    60   Input ~ 0
+Text HLabel 2900 2900 0    60   Input ~ 0
 SW1
-$Comp
-L 74LS245 U4
-U 1 1 4F81A8A5
-P 6350 2750
-F 0 "U4" H 6450 3325 60  0000 L BNN
-F 1 "74HC245" H 6400 2175 60  0000 L TNN
-	1    6350 2750
-	1    0    0    -1
-$EndComp
 $EndSCHEMATC

Commit message: Routing
Parts:
- added C26: 100n, symbol C
- added U10: 74HC165, symbol 74LS165
Connections:
- net +3.3V: now also C26.1, U10.16 (VCC)
- net BTNSHIFT_IN0: now also U10.10 (Ds)
- net BTN_CE: now also U10.15 (CE)
- net BTN_LOAD: now also U10.1 (Pl)
- net GND: now also C26.2, U10.8 (GND)
- net SHIFT_CLK: now also U10.2 (CP)
- net SW10: now also U10.12 (P1)
- net SW11: now also U10.13 (P2)
- net SW12: now also U10.14 (P3)
- net SW13: now also U10.3 (P4)
- net SW14: now also U10.4 (P5)
- net SW15: now also U10.5 (P6)
- net SW16: now also U10.6 (P7)
- net SW9: now also U10.11 (P0)
Changed lines of the file:
@@
-EESchema Schematic File Version 2  date Thu 19 Apr 2012 08:23:14 PM CEST
+EESchema Schematic File Version 2  date Thu 19 Apr 2012 10:08:52 PM CEST
 LIBS:power
 LIBS:device
@@
 $Descr A4 11700 8267
 encoding utf-8
-Sheet 2 5
+Sheet 3 6
 Title ""
 Date "19 apr 2012"
@@
 Comment4 ""
 $EndDescr
+Text HLabel 2550 4800 0    60   Input ~ 0
+BTNSHIFT_IN0
+Wire Wire Line
+	2900 4800 2550 4800
+Text HLabel 2650 5900 0    60   Input ~ 0
+SHIFT_CLK
+Text HLabel 2650 5750 0    60   Input ~ 0
+BTN_LOAD
+Text HLabel 2650 6000 0    60   Input ~ 0
+BTN_CE
+Wire Wire Line
+	2900 5900 2650 5900
+Wire Wire Line
+	2650 5750 2900 5750
+Wire Wire Line
+	2650 6000 2900 6000
+$Comp
+L C C26
+U 1 1 4F905CC6
+P 5150 5300
+F 0 "C26" H 5200 5400 50  0000 L CNN
+F 1 "100n" H 5200 5200 50  0000 L CNN
+	1    5150 5300
+	1    0    0    -1
+$EndComp
+$Comp
+L +3.3V #PWR024
+U 1 1 4F905CC5
+P 5150 4950
+F 0 "#PWR024" H 5150 4910 30  0001 C CNN
+F 1 "+3.3V" H 5150 5060 30  0000 C CNN
+	1    5150 4950
+	1    0    0    -1
+$EndComp
+$Comp
+L GND #PWR025
+U 1 1 4F905CC4
+P 5150 5700
+F 0 "#PWR025" H 5150 5700 30  0001 C CNN
+F 1 "GND" H 5150 5630 30  0001 C CNN
+	1    5150 5700
+	1    0    0    -1
+$EndComp
+Wire Wire Line
+	5150 5500 5150 5700
+Wire Wire Line
+	5150 4950 5150 5100
+$Comp
+L 74LS165 U10
+U 1 1 4F905CAB
+P 3600 5400
+F 0 "U10" H 3750 5350 60  0000 C CNN
+F 1 "74HC165" H 3750 5150 60  0000 C CNN
+	1    3600 5400
+	1    0    0    -1
+$EndComp
 NoConn ~ 4300 3000
 Wire Wire Line
@@
 $EndComp
 $Comp
-L GND #PWR03
+L GND #PWR026
 U 1 1 4F8DA672
 P 3300 4250
-F 0 "#PWR03" H 3300 4250 30  0001 C CNN
+F 0 "#PWR026" H 3300 4250 30  0001 C CNN
 F 1 "GND" H 3300 4180 30  0001 C CNN
 	1    3300 4250
@@
 $EndComp
 $Comp
-L +3.3V #PWR04
+L +3.3V #PWR027
 U 1 1 4F8DA671
 P 3300 2500
-F 0 "#PWR04" H 3300 2460 30  0001 C CNN
+F 0 "#PWR027" H 3300 2460 30  0001 C CNN
 F 1 "+3.3V" H 3300 2610 30  0000 C CNN
 	1    3300 2500
@@
 BTNSHIFT_IN0
 $Comp
-L GND #PWR05
+L GND #PWR028
 U 1 1 4F82A012
 P 5150 3850
-F 0 "#PWR05" H 5150 3850 30  0001 C CNN
+F 0 "#PWR028" H 5150 3850 30  0001 C CNN
 F 1 "GND" H 5150 3780 30  0001 C CNN
 	1    5150 3850
@@
 $EndComp
 $Comp
-L +3.3V #PWR06
+L +3.3V #PWR029
 U 1 1 4F82A00E
 P 5150 3100
-F 0 "#PWR06" H 5150 3060 30  0001 C CNN
+F 0 "#PWR029" H 5150 3060 30  0001 C CNN
 F 1 "+3.3V" H 5150 3210 30  0000 C CNN
 	1    5150 3100
@@
 	1    0    0    -1
 $EndComp
-Text HLabel 7200 3850 0    60   Input ~ 0
+Text HLabel 2900 5600 0    60   Input ~ 0
 SW16
-Text HLabel 7200 3750 0    60   Input ~ 0
+Text HLabel 2900 5500 0    60   Input ~ 0
 SW15
-Text HLabel 7200 3650 0    60   Input ~ 0
+Text HLabel 2900 5400 0    60   Input ~ 0
 SW14
-Text HLabel 7200 3550 0    60   Input ~ 0
+Text HLabel 2900 5300 0    60   Input ~ 0
 SW13
-Text HLabel 7200 3450 0    60   Input ~ 0
+Text HLabel 2900 5200 0    60   Input ~ 0
 SW12
-Text HLabel 7200 3350 0    60   Input ~ 0
+Text HLabel 2900 5100 0    60   Input ~ 0
 SW11
-Text HLabel 7200 3250 0    60   Input ~ 0
+Text HLabel 2900 5000 0    60   Input ~ 0
 SW10
-Text HLabel 7200 3150 0    60   Input ~ 0
+Text HLabel 2900 4900 0    60   Input ~ 0
 SW9
 Text HLabel 2900 3600 0    60   Input ~ 0
