File: encoders2.sch (KiCad schematic (older format))
At the start: 45 parts, among them U3 74HCT595, U8 74HC165

Commit message: Routing
Parts:
- removed C11, C6: 100n, symbol C
- removed C16: 10u, symbol C
- removed CK11, CK12, CK21, CK22, CK31, CK32, CK41, CK42: 10n, symbol C
- removed ENC1, ENC2, ENC3, ENC4: PEL12D, symbol PEL12D
- removed RK12, RK22, RK32, RK42: 390, symbol R
- removed RK13, RK23, RK33, RK43: 240, symbol R
- removed RK16, RK17, RK26, RK27, RK36, RK37, RK46, RK47, RPU1 (x4), RPU10, RPU11, RPU12, RPU5, RPU6, RPU7, RPU8, RPU9: 20k, symbol R
- removed U3: 74HCT595, symbol 74HC595-PWR
- removed U8: 74HC165, symbol 74LS165
- added C23, C25: 100n, symbol C
- added C24: 10u, symbol C
- added CK51, CK52, CK61, CK62, CK71, CK72, CK81, CK82: 10n, symbol C
- added ENC5, ENC6, ENC7, ENC8: PEL12D, symbol PEL12D
- added RK52, RK62, RK72, RK82: 390, symbol R
- added RK53, RK63, RK73, RK83: 240, symbol R
- added RK56, RK57, RK66, RK67, RK76, RK77, RK86, RK87, RPU13, RPU14, RPU15, RPU16, RPU17, RPU18, RPU19, RPU20, RPU21, RPU22, RPU23, RPU24: 20k, symbol R
- added U7: 74HCT595, symbol 74HC595-PWR
- added U9: 74HC165, symbol 74LS165
