File: encoders3.sch (KiCad schematic (older format))
At the start: 45 parts, among them U3 74HCT595, U8 74HC165

Commit message: Add last encoders
Parts:
- removed C11, C6: 100n, symbol C
- removed C16: 10u, symbol C
- removed CK11, CK12, CK21, CK22, CK31, CK32, CK41, CK42: 10n, symbol C
- removed ENC1, ENC2, ENC3, ENC4: PEL12D, symbol PEL12D
- removed RK12, RK22, RK32, RK42: 390, symbol R
- removed RK13, RK23, RK33, RK43: 240, symbol R
- removed RK16, RK17, RK26, RK27, RK36, RK37, RK46, RK47, RPU1 (x4), RPU10, RPU11, RPU12, RPU5, RPU6, RPU7, RPU8, RPU9: 20k, symbol R
- removed U3: 74HCT595, symbol 74HC595-PWR
- removed U8: 74HC165, symbol 74LS165
- added C30, C32: 100n, symbol C
- added C31: 10u, symbol C
- added CK101, CK102, CK111, CK112, CK121, CK122, CK91, CK92: 10n, symbol C
- added ENC10, ENC11, ENC12, ENC9: PEL12D, symbol PEL12D
- added RK102, RK112, RK122, RK92: 390, symbol R
- added RK103, RK113, RK123, RK93: 240, symbol R
- added RK106, RK107, RK116, RK117, RK126, RK127, RK96, RK97, RPU37, RPU38, RPU39, RPU40, RPU41, RPU42, RPU43, RPU44, RPU45, RPU46, RPU47, RPU48: 20k, symbol R
- added U13: 74HCT595, symbol 74HC595-PWR
- added U14: 74HC165, symbol 74LS165
