File: encoders4.sch (KiCad schematic (older format))
At the start: 45 parts, among them U3 74HCT595, U8 74HC165

Commit message: Add last encoders
Parts:
- removed C11, C6: 100n, symbol C
- removed C16: 10u, symbol C
- removed CK11, CK12, CK21, CK22, CK31, CK32, CK41, CK42: 10n, symbol C
- removed ENC1, ENC2, ENC3, ENC4: PEL12D, symbol PEL12D
- removed RK12, RK22, RK32, RK42: 390, symbol R
- removed RK13, RK23, RK33, RK43: 240, symbol R
- removed RK16, RK17, RK26, RK27, RK36, RK37, RK46, RK47, RPU1 (x4), RPU10, RPU11, RPU12, RPU5, RPU6, RPU7, RPU8, RPU9: 20k, symbol R
- removed U3: 74HCT595, symbol 74HC595-PWR
- removed U8: 74HC165, symbol 74LS165
- added C27, C29: 100n, symbol C
- added C28: 10u, symbol C
- added CK131, CK132, CK141, CK142, CK151, CK152, CK161, CK162: 10n, symbol C
- added ENC13, ENC14, ENC15, ENC16: PEL12D, symbol PEL12D
- added RK132, RK142, RK152, RK162: 390, symbol R
- added RK133, RK143, RK153, RK163: 240, symbol R
- added RK136, RK137, RK146, RK147, RK156, RK157, RK166, RK167, RPU25, RPU26, RPU27, RPU28, RPU29, RPU30, RPU31, RPU32, RPU33, RPU34, RPU35, RPU36: 20k, symbol R
- added U11: 74HCT595, symbol 74HC595-PWR
- added U12: 74HC165, symbol 74LS165
