File: io.sch (KiCad schematic (older format))
At the start: 15 parts, among them P1 MICROUSB, P3 DIN5, P4 DIN5, P6 CONN_5, P7 CONN_2, Q1 PDTA124X, Q2 PDTC123Y, U5 VOL617A

Commit message: Chaotic changes.
Parts:
- removed P6: CONN_5, symbol CONN_5
- removed P7: CONN_2, symbol CONN_2
- added P5: CONN_5, symbol CONN_5
- added Q4: PDTA124X, SOT23-3, symbol PDTA124X
- added Q5: PDTC123Y, SOT23-3, symbol PDTC123Y
- added R19: 20k, symbol R
- added R20, R21, R22: 220, symbol R
- added TP1, TP2, TP3, TP4, TP5, TP6, TP7, TP8: TST, symbol TST
- added U15: VOL617A, symbol OPTO-TRANSISTOR4
Connections:
- net labels added: MIDIIN2+, MIDIIN2-, MIDIOUT2+, MIDIOUT2-, MIDI_RX2, MIDI_TX2
- wire segments 39 -> 50
Other:
- note removed: "USB"
- moved on the sheet: P1, P3, P4, Q1, Q2, R10, R12, R13, R15, R16, R17, R8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

Commit message: Routing.
Parts:
- added TP13: TST, symbol TST
Connections:
- net +5V: now also TP2.1
- net GND: now also TP13.1
- net USB_5V: now also TP1.1
- net USB_DM: now also TP3.1
- net USB_DP: now also TP4.1
Changed lines of the file:
@@
-EESchema Schematic File Version 2  date Sun 05 May 2013 06:02:32 PM CEST
+EESchema Schematic File Version 2  date Wed 08 May 2013 08:54:31 PM CEST
 LIBS:power
 LIBS:device
@@
 $Descr A4 11700 8267
 encoding utf-8
-Sheet 4 10
+Sheet 5 10
 Title ""
-Date "5 may 2013"
+Date "8 may 2013"
 Rev ""
 Comp ""
@@
 Comment4 ""
 $EndDescr
+Connection ~ 9200 5200
+Connection ~ 10200 5000
+Connection ~ 9450 4150
+Wire Wire Line
+	9450 4250 9450 4100
+Wire Wire Line
+	9900 4100 9900 4250
+Wire Wire Line
+	4750 5550 4750 5200
+Wire Wire Line
+	4450 4900 4650 4900
+Wire Wire Line
+	2100 5350 2100 5200
+Wire Wire Line
+	2100 5200 2300 5200
+Wire Wire Line
+	2300 4900 1900 4900
+Wire Wire Line
+	2350 6650 2000 6650
+Wire Wire Line
+	3800 6400 4800 6400
+Wire Wire Line
+	3800 6400 3800 6150
+Wire Wire Line
+	3950 4900 3550 4900
+Wire Wire Line
+	5450 6100 5450 5950
+Wire Wire Line
+	5450 5950 5550 5950
+Wire Wire Line
+	2900 6300 3150 6300
+Wire Wire Line
+	1300 6300 1450 6300
+Wire Wire Line
+	2100 4800 2100 4900
+Connection ~ 2100 4900
+Wire Wire Line
+	3650 6300 4900 6300
+Wire Wire Line
+	4800 6400 4800 5750
+Wire Wire Line
+	4900 6300 4900 5850
+Wire Wire Line
+	4900 5850 5550 5850
+Wire Wire Line
+	4800 5750 5550 5750
+Wire Wire Line
+	4650 4900 4650 5650
+Wire Wire Line
+	4650 5650 5550 5650
+Wire Wire Line
+	4750 5550 5550 5550
+Wire Wire Line
+	4850 2750 3600 2750
+Wire Wire Line
+	9450 4750 9450 4800
+Connection ~ 2050 1350
+Wire Wire Line
+	2050 1250 2050 1350
+Wire Wire Line
+	1250 2750 1400 2750
+Wire Wire Line
+	2850 2750 3100 2750
+Wire Wire Line
+	4800 1250 4500 1250
+Wire Wire Line
+	4500 1250 4500 1650
+Wire Wire Line
+	4500 1650 3500 1650
+Wire Wire Line
+	4400 1350 4800 1350
+Wire Wire Line
+	4600 3250 4600 3050
+Wire Wire Line
+	4600 3050 4850 3050
+Wire Wire Line
+	8600 5100 9900 5100
+Connection ~ 9900 5000
+Wire Wire Line
+	9900 4750 9900 5000
+Wire Wire Line
+	10250 4900 8600 4900
+Wire Wire Line
+	9450 4800 8600 4800
+Wire Wire Line
+	8600 5200 9450 5200
+Wire Wire Line
+	9450 5200 9450 5400
+Wire Wire Line
+	10250 5000 8600 5000
+Wire Wire Line
+	3900 1350 3500 1350
+Wire Wire Line
+	3750 2600 3750 2850
+Wire Wire Line
+	3750 2850 4850 2850
+Wire Wire Line
+	2300 3100 1950 3100
+Wire Wire Line
+	2250 1350 1850 1350
+Wire Wire Line
+	2250 1650 2050 1650
+Wire Wire Line
+	2050 1650 2050 1800
+Wire Wire Line
+	4750 5200 3550 5200
+Connection ~ 10200 4900
+Connection ~ 9200 4800
+$Comp
+L TST TP13
+U 1 1 518940F0
+P 9200 5200
+F 0 "TP13" H 9200 5500 40  0000 C CNN
+F 1 "TST" H 9200 5450 30  0000 C CNN
+	1    9200 5200
+	-1   0    0    1
+$EndComp
 $Comp
 L TST TP8
@@
 	1    0    0    -1
 $EndComp
-Wire Wire Line
-	9900 4100 9900 4250
-Wire Wire Line
-	4750 5550 4750 5200
-Wire Wire Line
-	4450 4900 4650 4900
-Wire Wire Line
-	2100 5350 2100 5200
-Wire Wire Line
-	2100 5200 2300 5200
-Wire Wire Line
-	2300 4900 1900 4900
-Wire Wire Line
-	2350 6650 2000 6650
-Wire Wire Line
-	3800 6400 4800 6400
-Wire Wire Line
-	3800 6400 3800 6150
-Wire Wire Line
-	3950 4900 3550 4900
-Wire Wire Line
-	5450 6100 5450 5950
-Wire Wire Line
-	5450 5950 5550 5950
-Wire Wire Line
-	2900 6300 3150 6300
-Wire Wire Line
-	1300 6300 1450 6300
-Wire Wire Line
-	2100 4800 2100 4900
-Connection ~ 2100 4900
-Wire Wire Line
-	3650 6300 4900 6300
-Wire Wire Line
-	4800 6400 4800 5750
-Wire Wire Line
-	4900 6300 4900 5850
-Wire Wire Line
-	4900 5850 5550 5850
-Wire Wire Line
-	4800 5750 5550 5750
-Wire Wire Line
-	4650 4900 4650 5650
-Wire Wire Line
-	4650 5650 5550 5650
-Wire Wire Line
-	4750 5550 5550 5550
-Wire Wire Line
-	4850 2750 3600 2750
-Wire Wire Line
-	9450 4750 9450 4800
-Connection ~ 2050 1350
-Wire Wire Line
-	2050 1250 2050 1350
-Wire Wire Line
-	1250 2750 1400 2750
-Wire Wire Line
-	2850 2750 3100 2750
-Wire Wire Line
-	4800 1250 4500 1250
-Wire Wire Line
-	4500 1250 4500 1650
-Wire Wire Line
-	4500 1650 3500 1650
-Wire Wire Line
-	4400 1350 4800 1350
-Wire Wire Line
-	4600 3250 4600 3050
-Wire Wire Line
-	4600 3050 4850 3050
-Wire Wire Line
-	8600 5100 9900 5100
-Connection ~ 9900 5000
-Wire Wire Line
-	9900 4750 9900 5000
-Wire Wire Line
-	10250 4900 8600 4900
-Wire Wire Line
-	9450 4800 8600 4800
-Wire Wire Line
-	8600 5200 9450 5200
-Wire Wire Line
-	9450 5200 9450 5400
-Wire Wire Line
-	10250 5000 8600 5000
-Wire Wire Line
-	3900 1350 3500 1350
-Wire Wire Line
-	3750 2600 3750 2850
-Wire Wire Line
-	3750 2850 4850 2850
-Wire Wire Line
-	2300 3100 1950 3100
-Wire Wire Line
-	2250 1350 1850 1350
-Wire Wire Line
-	2250 1650 2050 1650
-Wire Wire Line
-	2050 1650 2050 1800
-Wire Wire Line
-	4750 5200 3550 5200
-Wire Wire Line
-	9450 4100 9450 4250
 $Comp
 L OPTO-TRANSISTOR4 U15
@@
 MIDI_TX2
 $Comp
-L +5V #PWR49
+L +5V #PWR038
 U 1 1 50CDE1D2
 P 3800 5650
-F 0 "#PWR49" H 3800 5740 20  0001 C CNN
+F 0 "#PWR038" H 3800 5740 20  0001 C CNN
 F 1 "+5V" H 3800 5740 30  0000 C CNN
 	1    3800 5650
@@
 $EndComp
 $Comp
-L GND #PWR51
+L GND #PWR039
 U 1 1 50CDE1CB
 P 5450 6100
-F 0 "#PWR51" H 5450 6100 30  0001 C CNN
+F 0 "#PWR039" H 5450 6100 30  0001 C CNN
 F 1 "GND" H 5450 6030 30  0001 C CNN
 	1    5450 6100
@@
 $EndComp
 $Comp
-L GND #PWR47
+L GND #PWR040
 U 1 1 50CDE1C9
 P 2900 7100
-F 0 "#PWR47" H 2900 7100 30  0001 C CNN
+F 0 "#PWR040" H 2900 7100 30  0001 C CNN
 F 1 "GND" H 2900 7030 30  0001 C CNN
 	1    2900 7100
@@
 $EndComp
 $Comp
-L +3.3V #PWR41
+L +3.3V #PWR041
 U 1 1 50CDE1C6
 P 2000 5850
-F 0 "#PWR41" H 2000 5810 30  0001 C CNN
+F 0 "#PWR041" H 2000 5810 30  0001 C CNN
 F 1 "+3.3V" H 2000 5960 30  0000 C CNN
 	1    2000 5850
@@
 $EndComp
 $Comp
-L GND #PWR45
+L GND #PWR042
 U 1 1 50CDE1C4
 P 2100 5350
-F 0 "#PWR45" H 2100 5350 30  0001 C CNN
+F 0 "#PWR042" H 2100 5350 30  0001 C CNN
 F 1 "GND" H 2100 5280 30  0001 C CNN
 	1    2100 5350
@@
 $EndComp
 $Comp
-L +3.3V #PWR44
+L +3.3V #PWR043
 U 1 1 50CDE1C3
 P 2100 4300
-F 0 "#PWR44" H 2100 4260 30  0001 C CNN
+F 0 "#PWR043" H 2100 4260 30  0001 C CNN
 F 1 "+3.3V" H 2100 4410 30  0000 C CNN
 	1    2100 4300
@@
 $EndComp
 $Comp
-L +3.3V #PWR42
+L +3.3V #PWR044
 U 1 1 4F8985F8
 P 2050 750
-F 0 "#PWR42" H 2050 710 30  0001 C CNN
+F 0 "#PWR044" H 2050 710 30  0001 C CNN
 F 1 "+3.3V" H 2050 860 30  0000 C CNN
 	1    2050 750
@@
 $EndComp
 $Comp
-L GND #PWR43
+L GND #PWR045
 U 1 1 4F8984E9
 P 2050 1800
-F 0 "#PWR43" H 2050 1800 30  0001 C CNN
+F 0 "#PWR045" H 2050 1800 30  0001 C CNN
 F 1 "GND" H 2050 1730 30  0001 C CNN
 	1    2050 1800
@@
 $EndComp
 $Comp
-L +3.3V #PWR40
+L +3.3V #PWR046
 U 1 1 4F898360
 P 1950 2300
-F 0 "#PWR40" H 1950 2260 30  0001 C CNN
+F 0 "#PWR046" H 1950 2260 30  0001 C CNN
 F 1 "+3.3V" H 1950 2410 30  0000 C CNN
 	1    1950 2300
@@
 $EndComp
 $Comp
-L GND #PWR46
+L GND #PWR047
 U 1 1 4F897803
 P 2850 3550
-F 0 "#PWR46" H 2850 3550 30  0001 C CNN
+F 0 "#PWR047" H 2850 3550 30  0001 C CNN
 F 1 "GND" H 2850 3480 30  0001 C CNN
 	1    2850 3550
@@
 $EndComp
 $Comp
-L GND #PWR50
+L GND #PWR048
 U 1 1 4F896A83
 P 4600 3250
-F 0 "#PWR50" H 4600 3250 30  0001 C CNN
+F 0 "#PWR048" H 4600 3250 30  0001 C CNN
 F 1 "GND" H 4600 3180 30  0001 C CNN
 	1    4600 3250
@@
 $EndComp
 $Comp
-L +5V #PWR48
+L +5V #PWR049
 U 1 1 4F8968A2
 P 3750 2100
-F 0 "#PWR48" H 3750 2190 20  0001 C CNN
+F 0 "#PWR049" H 3750 2190 20  0001 C CNN
 F 1 "+5V" H 3750 2190 30  0000 C CNN
 	1    3750 2100
@@
 $EndComp
 $Comp
-L GND #PWR55
+L GND #PWR050
 U 1 1 4F894AD1
 P 9900 5600
-F 0 "#PWR55" H 9900 5600 30  0001 C CNN
+F 0 "#PWR050" H 9900 5600 30  0001 C CNN
 F 1 "GND" H 9900 5530 30  0001 C CNN
 	1    9900 5600
@@
 $EndComp
 $Comp
-L +3.3V #PWR54
+L +3.3V #PWR051
 U 1 1 4F89446F
 P 9900 4100
-F 0 "#PWR54" H 9900 4060 30  0001 C CNN
+F 0 "#PWR051" H 9900 4060 30  0001 C CNN
 F 1 "+3.3V" H 9900 4210 30  0000 C CNN
 	1    9900 4100
@@
 $EndComp
 $Comp
-L GND #PWR53
+L GND #PWR052
 U 1 1 4F894376
 P 9450 5400
-F 0 "#PWR53" H 9450 5400 30  0001 C CNN
+F 0 "#PWR052" H 9450 5400 30  0001 C CNN
 F 1 "GND" H 9450 5330 30  0001 C CNN
 	1    9450 5400
@@
 $EndComp
 $Comp
-L +5V #PWR52
+L +5V #PWR053
 U 1 1 4F894373
 P 9450 4100
-F 0 "#PWR52" H 9450 4190 20  0001 C CNN
+F 0 "#PWR053" H 9450 4190 20  0001 C CNN
 F 1 "+5V" H 9450 4190 30  0000 C CNN
 	1    9450 4100

Commit message: Layouting.
Connections:
- net MIDI_RX: now also TP5.1
- net MIDI_RX2: now also TP7.1
- net MIDI_TX: now also TP6.1
- net MIDI_TX2: now also TP8.1
Changed lines of the file:
@@
-EESchema Schematic File Version 2  date Wed 08 May 2013 08:54:31 PM CEST
+EESchema Schematic File Version 2  date Sun 19 May 2013 11:54:05 AM CEST
 LIBS:power
 LIBS:device
@@
 Sheet 5 10
 Title ""
-Date "8 may 2013"
+Date "19 may 2013"
 Rev ""
 Comp ""
@@
 Comment4 ""
 $EndDescr
+Connection ~ 2000 4900
+Connection ~ 1400 6300
+Connection ~ 1950 1350
+Connection ~ 1950 1350
+Connection ~ 1350 2750
 Connection ~ 9200 5200
 Connection ~ 10200 5000
@@
 MIDI_TX2
 $Comp
-L +5V #PWR038
+L +5V #PWR037
 U 1 1 50CDE1D2
 P 3800 5650
-F 0 "#PWR038" H 3800 5740 20  0001 C CNN
+F 0 "#PWR037" H 3800 5740 20  0001 C CNN
 F 1 "+5V" H 3800 5740 30  0000 C CNN
 	1    3800 5650
@@
 $EndComp
 $Comp
-L GND #PWR039
+L GND #PWR038
 U 1 1 50CDE1CB
 P 5450 6100
-F 0 "#PWR039" H 5450 6100 30  0001 C CNN
+F 0 "#PWR038" H 5450 6100 30  0001 C CNN
 F 1 "GND" H 5450 6030 30  0001 C CNN
 	1    5450 6100
@@
 $EndComp
 $Comp
-L GND #PWR040
+L GND #PWR039
 U 1 1 50CDE1C9
 P 2900 7100
-F 0 "#PWR040" H 2900 7100 30  0001 C CNN
+F 0 "#PWR039" H 2900 7100 30  0001 C CNN
 F 1 "GND" H 2900 7030 30  0001 C CNN
 	1    2900 7100
@@
 $EndComp
 $Comp
-L +3.3V #PWR041
+L +3.3V #PWR040
 U 1 1 50CDE1C6
 P 2000 5850
-F 0 "#PWR041" H 2000 5810 30  0001 C CNN
+F 0 "#PWR040" H 2000 5810 30  0001 C CNN
 F 1 "+3.3V" H 2000 5960 30  0000 C CNN
 	1    2000 5850
@@
 $EndComp
 $Comp
-L GND #PWR042
+L GND #PWR041
 U 1 1 50CDE1C4
 P 2100 5350
-F 0 "#PWR042" H 2100 5350 30  0001 C CNN
+F 0 "#PWR041" H 2100 5350 30  0001 C CNN
 F 1 "GND" H 2100 5280 30  0001 C CNN
 	1    2100 5350
@@
 $EndComp
 $Comp
-L +3.3V #PWR043
+L +3.3V #PWR042
 U 1 1 50CDE1C3
 P 2100 4300
-F 0 "#PWR043" H 2100 4260 30  0001 C CNN
+F 0 "#PWR042" H 2100 4260 30  0001 C CNN
 F 1 "+3.3V" H 2100 4410 30  0000 C CNN
 	1    2100 4300
@@
 $EndComp
 $Comp
-L +3.3V #PWR044
+L +3.3V #PWR043
 U 1 1 4F8985F8
 P 2050 750
-F 0 "#PWR044" H 2050 710 30  0001 C CNN
+F 0 "#PWR043" H 2050 710 30  0001 C CNN
 F 1 "+3.3V" H 2050 860 30  0000 C CNN
 	1    2050 750
@@
 $EndComp
 $Comp
-L GND #PWR045
+L GND #PWR044
 U 1 1 4F8984E9
 P 2050 1800
-F 0 "#PWR045" H 2050 1800 30  0001 C CNN
+F 0 "#PWR044" H 2050 1800 30  0001 C CNN
 F 1 "GND" H 2050 1730 30  0001 C CNN
 	1    2050 1800
@@
 $EndComp
 $Comp
-L +3.3V #PWR046
+L +3.3V #PWR045
 U 1 1 4F898360
 P 1950 2300
-F 0 "#PWR046" H 1950 2260 30  0001 C CNN
+F 0 "#PWR045" H 1950 2260 30  0001 C CNN
 F 1 "+3.3V" H 1950 2410 30  0000 C CNN
 	1    1950 2300
@@
 $EndComp
 $Comp
-L GND #PWR047
+L GND #PWR046
 U 1 1 4F897803
 P 2850 3550
-F 0 "#PWR047" H 2850 3550 30  0001 C CNN
+F 0 "#PWR046" H 2850 3550 30  0001 C CNN
 F 1 "GND" H 2850 3480 30  0001 C CNN
 	1    2850 3550
@@
 $EndComp
 $Comp
-L GND #PWR048
+L GND #PWR047
 U 1 1 4F896A83
 P 4600 3250
-F 0 "#PWR048" H 4600 3250 30  0001 C CNN
+F 0 "#PWR047" H 4600 3250 30  0001 C CNN
 F 1 "GND" H 4600 3180 30  0001 C CNN
 	1    4600 3250
@@
 $EndComp
 $Comp
-L +5V #PWR049
+L +5V #PWR048
 U 1 1 4F8968A2
 P 3750 2100
-F 0 "#PWR049" H 3750 2190 20  0001 C CNN
+F 0 "#PWR048" H 3750 2190 20  0001 C CNN
 F 1 "+5V" H 3750 2190 30  0000 C CNN
 	1    3750 2100
@@
 $EndComp
 $Comp
-L GND #PWR050
+L GND #PWR049
 U 1 1 4F894AD1
 P 9900 5600
-F 0 "#PWR050" H 9900 5600 30  0001 C CNN
+F 0 "#PWR049" H 9900 5600 30  0001 C CNN
 F 1 "GND" H 9900 5530 30  0001 C CNN
 	1    9900 5600
@@
 $EndComp
 $Comp
-L +3.3V #PWR051
+L +3.3V #PWR050
 U 1 1 4F89446F
 P 9900 4100
-F 0 "#PWR051" H 9900 4060 30  0001 C CNN
+F 0 "#PWR050" H 9900 4060 30  0001 C CNN
 F 1 "+3.3V" H 9900 4210 30  0000 C CNN
 	1    9900 4100
@@
 $EndComp
 $Comp
-L GND #PWR052
+L GND #PWR051
 U 1 1 4F894376
 P 9450 5400
-F 0 "#PWR052" H 9450 5400 30  0001 C CNN
+F 0 "#PWR051" H 9450 5400 30  0001 C CNN
 F 1 "GND" H 9450 5330 30  0001 C CNN
 	1    9450 5400
@@
 $EndComp
 $Comp
-L +5V #PWR053
+L +5V #PWR052
 U 1 1 4F894373
 P 9450 4100
-F 0 "#PWR053" H 9450 4190 20  0001 C CNN
+F 0 "#PWR052" H 9450 4190 20  0001 C CNN
 F 1 "+5V" H 9450 4190 30  0000 C CNN
 	1    9450 4100

Commit message: Routing.
Connections:
- net +3.3V: no longer R19.2, R8.2
- new net VPULLUP: R19.2, R8.2
Other:
- note added: "mount 1k5 according to errata?"
Changed lines of the file:
@@
-EESchema Schematic File Version 2  date Sun 19 May 2013 11:54:05 AM CEST
+EESchema Schematic File Version 2  date Sun 26 May 2013 03:42:57 PM CEST
 LIBS:power
 LIBS:device
@@
 Sheet 5 10
 Title ""
-Date "19 may 2013"
+Date "26 may 2013"
 Rev ""
 Comp ""
@@
 Comment4 ""
 $EndDescr
+Wire Wire Line
+	2100 4300 2400 4300
 Connection ~ 2000 4900
 Connection ~ 1400 6300
@@
 Connection ~ 10200 4900
 Connection ~ 9200 4800
+Wire Wire Line
+	2050 750  2350 750
+Text GLabel 2400 4300 2    60   Input ~ 0
+VPULLUP
+Text GLabel 2350 750  2    60   Input ~ 0
+VPULLUP
+Text Notes 1450 4450 0    60   ~ 0
+mount 1k5 according to errata?
+Text Notes 1400 900  0    60   ~ 0
+mount 1k5 according to errata?
 $Comp
 L TST TP13
@@
 F 1 "GND" H 2100 5280 30  0001 C CNN
 	1    2100 5350
-	1    0    0    -1
-$EndComp
-$Comp
-L +3.3V #PWR042
-U 1 1 50CDE1C3
-P 2100 4300
-F 0 "#PWR042" H 2100 4260 30  0001 C CNN
-F 1 "+3.3V" H 2100 4410 30  0000 C CNN
-	1    2100 4300
 	1    0    0    -1
 $EndComp
@@
 	1    0    0    -1
 $EndComp
-$Comp
-L +3.3V #PWR043
-U 1 1 4F8985F8
-P 2050 750
-F 0 "#PWR043" H 2050 710 30  0001 C CNN
-F 1 "+3.3V" H 2050 860 30  0000 C CNN
-	1    2050 750
-	1    0    0    -1
-$EndComp

Commit message: Finished board CAD?
Parts:
- added D5, D6, D7, D8: LED, symbol LED
- added R18, R26, R27, R28: 390, symbol R
Connections:
- net +3.3V: now also D5.1 (A), D6.1 (A), D7.1 (A), D8.1 (A)
- net MIDI_RX: now also R18.2
- net MIDI_RX2: now also R27.2
- net at Q2.3 (C), R15.2: now also R26.2
- net at Q5.3 (C), R20.2: now also R28.2
- new net: D6.2 (K), R26.1
- new net: D5.2 (K), R18.1
- new net: D7.2 (K), R27.1
- new net: D8.2 (K), R28.1
Other:
- moved on the sheet: P3, P4, Q1, Q2, R15, R16, R17, R8, TP5, TP6, U5
