File: panel.sch (KiCad schematic (older format))
At the start: 34 parts, among them Q3 PDTC123Y, SW1 101-0661-EV, SW2 101-0661-EV, SW3 101-0661-EV, SW4 101-0661-EV, SW5 101-0661-EV

Commit message: Layouting.
Parts:
- removed C19: 100n, symbol C
- removed CK1, CK2: DNP, symbol C
Connections:
- net BL-: now reaches LCD1.13 (C2-), LCD1.2 (C1-), Q3.3 (C)
- net BL+: now reaches LCD1.1 (A1+), LCD1.14 (A2+), R6.1
Changed lines of the file:
@@
-EESchema Schematic File Version 2  date Wed 08 May 2013 08:54:31 PM CEST
+EESchema Schematic File Version 2  date Sun 19 May 2013 11:54:05 AM CEST
 LIBS:power
 LIBS:device
@@
 Sheet 2 10
 Title ""
-Date "8 may 2013"
+Date "19 may 2013"
 Rev ""
 Comp ""
@@
 Comment4 ""
 $EndDescr
+Text Label 2950 5450 0    60   ~ 0
+BL+
+Text Label 2700 5750 0    60   ~ 0
+BL-
 Connection ~ 6400 3300
 Wire Wire Line
@@
 Wire Wire Line
 	5000 3900 5000 3950
-Connection ~ 7000 4000
-Wire Wire Line
-	7000 4000 7000 4300
 Wire Wire Line
 	6600 3300 6600 3350
@@
 	4800 1550 4800 1600
 Wire Wire Line
-	5200 6600 4950 6600
-Wire Wire Line
 	4950 6150 4950 6200
 Wire Wire Line
@@
 Wire Wire Line
 	4950 6600 4950 6650
-Wire Wire Line
-	4950 6200 5200 6200
 Connection ~ 9000 2200
 Wire Wire Line
@@
 Connection ~ 4700 2500
 Wire Wire Line
-	7000 4700 7300 4700
-Wire Wire Line
-	7150 4750 7150 4700
-Connection ~ 7150 4700
-Wire Wire Line
 	7700 4200 6250 4200
 Wire Wire Line
@@
 Wire Wire Line
 	6400 3850 6400 4000
-Wire Wire Line
-	7300 4300 7300 4200
-Connection ~ 7300 4200
 Wire Wire Line
 	6250 4000 7700 4000
@@
 F 1 "PEL12D" H 5700 4350 60  0000 C CNN
 	1    5700 4100
-	1    0    0    -1
-$EndComp
-$Comp
-L GND #PWR04
-U 1 1 51867E31
-P 7150 4750
-F 0 "#PWR04" H 7150 4750 30  0001 C CNN
-F 1 "GND" H 7150 4680 30  0001 C CNN
-	1    7150 4750
-	1    0    0    -1
-$EndComp
-$Comp
-L C CK2
-U 1 1 51867E30
-P 7300 4500
-F 0 "CK2" H 7350 4600 50  0000 L CNN
-F 1 "DNP" H 7350 4400 50  0000 L CNN
-	1    7300 4500
-	1    0    0    -1
-$EndComp
-$Comp
-L C CK1
-U 1 1 51867E2F
-P 7000 4500
-F 0 "CK1" H 7050 4600 50  0000 L CNN
-F 1 "DNP" H 7050 4400 50  0000 L CNN
-	1    7000 4500
 	1    0    0    -1
 $EndComp
@@
 BTN1
 $Comp
-L +3.3V #PWR05
+L +3.3V #PWR04
 U 1 1 50CC7FBF
 P 3800 6850
-F 0 "#PWR05" H 3800 6810 30  0001 C CNN
+F 0 "#PWR04" H 3800 6810 30  0001 C CNN
 F 1 "+3.3V" H 3800 6960 30  0000 C CNN
 	1    3800 6850
@@
 LCD_A0
 $Comp
-L GND #PWR06
+L GND #PWR05
 U 1 1 50CC7FBE
 P 2600 6550
-F 0 "#PWR06" H 2600 6550 30  0001 C CNN
+F 0 "#PWR05" H 2600 6550 30  0001 C CNN
 F 1 "GND" H 2600 6480 30  0001 C CNN
 	1    2600 6550
@@
 $EndComp
 $Comp
-L +5V #PWR07
+L +5V #PWR06
 U 1 1 50CC7FBB
 P 2150 5450
-F 0 "#PWR07" H 2150 5540 20  0001 C CNN
+F 0 "#PWR06" H 2150 5540 20  0001 C CNN
 F 1 "+5V" H 2150 5540 30  0000 C CNN
 	1    2150 5450
@@
 Backlight at 5V, 80mA, Vf=2.2V --> 35ohm (0.25W),\nignoring drop in transistor. Base resistor\ncould be about 5k.
 $Comp
-L GND #PWR08
+L GND #PWR07
 U 1 1 50CC7FBA
 P 4500 6650
-F 0 "#PWR08" H 4500 6650 30  0001 C CNN
+F 0 "#PWR07" H 4500 6650 30  0001 C CNN
 F 1 "GND" H 4500 6580 30  0001 C CNN
 	1    4500 6650
@@
 $EndComp
 $Comp
-L +3.3V #PWR09
+L +3.3V #PWR08
 U 1 1 50CC7FB9
 P 4300 6600
-F 0 "#PWR09" H 4300 6560 30  0001 C CNN
+F 0 "#PWR08" H 4300 6560 30  0001 C CNN
 F 1 "+3.3V" H 4300 6710 30  0000 C CNN
 	1    4300 6600
@@
 $EndComp
 $Comp
-L GND #PWR010
+L GND #PWR09
 U 1 1 50CC7FB5
 P 6100 6100
-F 0 "#PWR010" H 6100 6100 30  0001 C CNN
+F 0 "#PWR09" H 6100 6100 30  0001 C CNN
 F 1 "GND" H 6100 6030 30  0001 C CNN
 	1    6100 6100
@@
 $EndComp
 $Comp
-L +3.3V #PWR011
+L +3.3V #PWR010
 U 1 1 50CC7FB3
 P 4950 6150
-F 0 "#PWR011" H 4950 6110 30  0001 C CNN
+F 0 "#PWR010" H 4950 6110 30  0001 C CNN
 F 1 "+3.3V" H 4950 6260 30  0000 C CNN
 	1    4950 6150
@@
 $EndComp
 $Comp
-L GND #PWR012
+L GND #PWR011
 U 1 1 50CC7FB2
 P 4950 6650
-F 0 "#PWR012" H 4950 6650 30  0001 C CNN
+F 0 "#PWR011" H 4950 6650 30  0001 C CNN
 F 1 "GND" H 4950 6580 30  0001 C CNN
 	1    4950 6650
@@
 $EndComp
 $Comp
-L C C19
-U 1 1 50CC7FB0
-P 5200 6400
-F 0 "C19" H 5250 6500 50  0000 L CNN
-F 1 "100n" H 5250 6300 50  0000 L CNN
-	1    5200 6400
-	1    0    0    -1
-$EndComp
-$Comp
 L R R1
 U 1 1 50CC7EBD
@@
 $EndComp
 $Comp
-L GND #PWR013
+L GND #PWR012
 U 1 1 50CC7EB9
 P 3700 2650
-F 0 "#PWR013" H 3700 2650 30  0001 C CNN
+F 0 "#PWR012" H 3700 2650 30  0001 C CNN
 F 1 "GND" H 3700 2580 30  0001 C CNN
 	1    3700 2650
@@
 $EndComp
 $Comp
-L +3.3V #PWR014
+L +3.3V #PWR013
 U 1 1 50CC7EB8
 P 4950 1000
-F 0 "#PWR014" H 4950 960 30  0001 C CNN
+F 0 "#PWR013" H 4950 960 30  0001 C CNN
 F 1 "+3.3V" H 4950 1110 30  0000 C CNN
 	1    4950 1000
@@
 BTN5
 $Comp
-L +3.3V #PWR015
+L +3.3V #PWR014
 U 1 1 50CC7EAC
 P 9000 1050
-F 0 "#PWR015" H 9000 1010 30  0001 C CNN
+F 0 "#PWR014" H 9000 1010 30  0001 C CNN
 F 1 "+3.3V" H 9000 1160 30  0000 C CNN
 	1    9000 1050

Commit message: Finished board CAD?
Parts:
- added DS1, DS2, DS3, DS4: LED, symbol LED
- R6: value 35 -> 36
Connections:
- net +3.3V: now also DS1.1 (A), DS2.1 (A), DS3.1 (A), DS4.1 (A)
- net at D4.2 (K), R14.1: now also DS4.2 (K)
- net at D3.2 (K), R11.1: now also DS3.2 (K)
- net at D2.2 (K), R9.1: now also DS2.2 (K)
- net at D1.2 (K), R7.1: now also DS1.2 (K)
Other:
- moved on the sheet: D1, D2, D3, D4, R11, R14, R7, R9

Commit message: Connect display RST to VPULLUP. Fix silkscreen.
Connections:
- net +3.3V: no longer LCD1.27 (RST)
- new net LCD_RST: LCD1.27 (RST)
Changed lines of the file:
@@
-EESchema Schematic File Version 2  date Sat 08 Jun 2013 06:16:56 PM CEST
+EESchema Schematic File Version 2  date Sun 09 Jun 2013 01:05:06 PM CEST
 LIBS:power
 LIBS:device
@@
 Sheet 2 10
 Title ""
-Date "8 jun 2013"
+Date "9 jun 2013"
 Rev ""
 Comp ""
@@
 Comment4 ""
 $EndDescr
+Text HLabel 3800 6850 3    60   Input ~ 0
+LCD_RST
 Wire Wire Line
 	10150 800  10150 2850
@@
 Text HLabel 4700 1250 1    60   Output ~ 0
 BTN1
-$Comp
-L +3.3V #PWR04
-U 1 1 50CC7FBF
-P 3800 6850
-F 0 "#PWR04" H 3800 6810 30  0001 C CNN
-F 1 "+3.3V" H 3800 6960 30  0000 C CNN
-	1    3800 6850
-	-1   0    0    1
-$EndComp
 Text Label 3700 6850 1    60   ~ 0
 CS_LCD
@@
 LCD_A0
 $Comp
-L GND #PWR05
+L GND #PWR04
 U 1 1 50CC7FBE
 P 2600 6550
-F 0 "#PWR05" H 2600 6550 30  0001 C CNN
+F 0 "#PWR04" H 2600 6550 30  0001 C CNN
 F 1 "GND" H 2600 6480 30  0001 C CNN
 	1    2600 6550
@@
 $EndComp
 $Comp
-L +5V #PWR06
+L +5V #PWR05
 U 1 1 50CC7FBB
 P 2150 5450
-F 0 "#PWR06" H 2150 5540 20  0001 C CNN
+F 0 "#PWR05" H 2150 5540 20  0001 C CNN
 F 1 "+5V" H 2150 5540 30  0000 C CNN
 	1    2150 5450
@@
 Backlight at 5V, 80mA, Vf=2.2V --> 35ohm (0.25W),\nignoring drop in transistor. Base resistor\ncould be about 5k.
 $Comp
-L GND #PWR07
+L GND #PWR06
 U 1 1 50CC7FBA
 P 4500 6650
-F 0 "#PWR07" H 4500 6650 30  0001 C CNN
+F 0 "#PWR06" H 4500 6650 30  0001 C CNN
 F 1 "GND" H 4500 6580 30  0001 C CNN
 	1    4500 6650
@@
 $EndComp
 $Comp
-L +3.3V #PWR08
+L +3.3V #PWR07
 U 1 1 50CC7FB9
 P 4300 6600
-F 0 "#PWR08" H 4300 6560 30  0001 C CNN
+F 0 "#PWR07" H 4300 6560 30  0001 C CNN
 F 1 "+3.3V" H 4300 6710 30  0000 C CNN
 	1    4300 6600
@@
 $EndComp
 $Comp
-L GND #PWR09
+L GND #PWR08
 U 1 1 50CC7FB5
 P 6100 6100
-F 0 "#PWR09" H 6100 6100 30  0001 C CNN
+F 0 "#PWR08" H 6100 6100 30  0001 C CNN
 F 1 "GND" H 6100 6030 30  0001 C CNN
 	1    6100 6100
@@
 $EndComp
 $Comp
-L +3.3V #PWR010
+L +3.3V #PWR09
 U 1 1 50CC7FB3
 P 4950 6150
-F 0 "#PWR010" H 4950 6110 30  0001 C CNN
+F 0 "#PWR09" H 4950 6110 30  0001 C CNN
 F 1 "+3.3V" H 4950 6260 30  0000 C CNN
 	1    4950 6150
@@
 $EndComp
 $Comp
-L GND #PWR011
+L GND #PWR010
 U 1 1 50CC7FB2
 P 4950 6650
-F 0 "#PWR011" H 4950 6650 30  0001 C CNN
+F 0 "#PWR010" H 4950 6650 30  0001 C CNN
 F 1 "GND" H 4950 6580 30  0001 C CNN
 	1    4950 6650
@@
 $EndComp
 $Comp
-L GND #PWR012
+L GND #PWR011
 U 1 1 50CC7EB9
 P 3700 2650
-F 0 "#PWR012" H 3700 2650 30  0001 C CNN
+F 0 "#PWR011" H 3700 2650 30  0001 C CNN
 F 1 "GND" H 3700 2580 30  0001 C CNN
 	1    3700 2650
@@
 $EndComp
 $Comp
-L +3.3V #PWR013
+L +3.3V #PWR012
 U 1 1 50CC7EB8
 P 4950 1000
-F 0 "#PWR013" H 4950 960 30  0001 C CNN
+F 0 "#PWR012" H 4950 960 30  0001 C CNN
 F 1 "+3.3V" H 4950 1110 30  0000 C CNN
 	1    4950 1000
@@
 BTN5
 $Comp
-L +3.3V #PWR014
+L +3.3V #PWR013
 U 1 1 50CC7EAC
 P 10150 800
-F 0 "#PWR014" H 10150 760 30  0001 C CNN
+F 0 "#PWR013" H 10150 760 30  0001 C CNN
 F 1 "+3.3V" H 10150 910 30  0000 C CNN
 	1    10150 800
